File: hardware/pcb/24-c-rtc-memory.sch (KiCad schematic (older format))
At the start: 7 parts, among them U701 24LC512, U702 DS1307+, Y701 CRYSTAL-32.768KHZSMD-3.2X1.5

Commit message: Changed uC
Parts:
- Y701: symbol SparkFun-Clocks:CRYSTAL-32.768KHZSMD-3.2X1.5 -> 24-clocks-rescue:CRYSTAL-32.768KHZSMD-3.2X1.5-SparkFun-Clocks
Changed lines of the file:
@@
 EESchema Schematic File Version 4
-LIBS:24-clocks-cache
-EELAYER 29 0
+EELAYER 30 0
 EELAYER END
 $Descr A4 11693 8268
@@
 	6600 4850 6600 4950
 $Comp
-L SparkFun-Clocks:CRYSTAL-32.768KHZSMD-3.2X1.5 Y701
+L 24-clocks-rescue:CRYSTAL-32.768KHZSMD-3.2X1.5-SparkFun-Clocks Y701
 U 1 1 5FD418B6
 P 5200 5300
+AR Path="/5FD418B6" Ref="Y701"  Part="1"
+AR Path="/5FDBDABC/5FD418B6" Ref="Y701"  Part="1"
 F 0 "Y701" V 5105 5398 45  0000 L CNN
 F 1 "CRYSTAL-32.768KHZSMD-3.2X1.5" V 5189 5398 45  0000 L CNN

Commit message: Updated processor pins and added testpoints
Parts:
- added TP701: I2C-SDA, symbol Connector:TestPoint
- added TP702: I2C-SCL, symbol Connector:TestPoint
Connections:
- net I2C-SCL: now also TP702.1
- net I2C-SDA: now also TP701.1
Changed lines of the file:
@@
 	0    1    1    0
 $EndComp
+$Comp
+L Connector:TestPoint TP701
+U 1 1 5FF95498
+P 3850 1000
+F 0 "TP701" H 3900 1100 50  0000 L CNN
+F 1 "I2C-SDA" H 3908 1027 50  0001 L CNN
+F 2 "" H 4050 1000 50  0001 C CNN
+F 3 "~" H 4050 1000 50  0001 C CNN
+	1    3850 1000
+	-1   0    0    -1
+$EndComp
+$Comp
+L Connector:TestPoint TP702
+U 1 1 5FF96021
+P 4000 1000
+F 0 "TP702" H 4050 1100 50  0000 L CNN
+F 1 "I2C-SCL" H 4058 1027 50  0001 L CNN
+F 2 "" H 4200 1000 50  0001 C CNN
+F 3 "~" H 4200 1000 50  0001 C CNN
+	1    4000 1000
+	1    0    0    -1
+$EndComp
+Wire Wire Line
+	4000 1000 4000 1100
+Wire Wire Line
+	3850 1000 3850 1250
 $EndSCHEMATC

Commit message: Small changes
Parts:
- added TP703: RC2032, symbol Connector:TestPoint
- BT701: value Battery_Cell -> RC2032
Connections:
- net at BT701.1 (+), U702.3 (VBAT): now also TP703.1
Other:
- moved on the sheet: C702
Changed lines of the file:
@@
 EESchema Schematic File Version 4
-EELAYER 30 0
+LIBS:24-clocks-cache
+EELAYER 29 0
 EELAYER END
 $Descr A4 11693 8268
@@
 L Device:C C702
 U 1 1 5FDCBDFD
-P 4350 5150
-F 0 "C702" H 4465 5196 50  0000 L CNN
-F 1 "100nF" H 4465 5105 50  0000 L CNN
-F 2 "C0603" H 4388 5000 50  0001 C CNN
-F 3 "~" H 4350 5150 50  0001 C CNN
-F 4 "-SLAVE" H 4350 5150 50  0001 C CNN "Config"
-	1    4350 5150
+P 3650 5100
+F 0 "C702" H 3765 5146 50  0000 L CNN
+F 1 "100nF" H 3765 5055 50  0000 L CNN
+F 2 "C0603" H 3688 4950 50  0001 C CNN
+F 3 "~" H 3650 5100 50  0001 C CNN
+F 4 "-SLAVE" H 3650 5100 50  0001 C CNN "Config"
+	1    3650 5100
 	1    0    0    -1
 $EndComp
@@
 L power:GND #PWR0710
 U 1 1 5FDCBE03
-P 4350 5350
-F 0 "#PWR0710" H 4350 5100 50  0001 C CNN
-F 1 "GND" H 4355 5177 50  0000 C CNN
-F 2 "" H 4350 5350 50  0001 C CNN
-F 3 "" H 4350 5350 50  0001 C CNN
-	1    4350 5350
+P 3650 5300
+F 0 "#PWR0710" H 3650 5050 50  0001 C CNN
+F 1 "GND" H 3655 5127 50  0000 C CNN
+F 2 "" H 3650 5300 50  0001 C CNN
+F 3 "" H 3650 5300 50  0001 C CNN
+	1    3650 5300
 	1    0    0    -1
 $EndComp
@@
 L power:+3V3 #PWR0707
 U 1 1 5FDCBE09
-P 4350 4950
-F 0 "#PWR0707" H 4350 4800 50  0001 C CNN
-F 1 "+3V3" H 4365 5123 50  0000 C CNN
-F 2 "" H 4350 4950 50  0001 C CNN
-F 3 "" H 4350 4950 50  0001 C CNN
-	1    4350 4950
-	1    0    0    -1
-$EndComp
-Wire Wire Line
-	4350 4950 4350 5000
-Wire Wire Line
-	4350 5300 4350 5350
+P 3650 4900
+F 0 "#PWR0707" H 3650 4750 50  0001 C CNN
+F 1 "+3V3" H 3665 5073 50  0000 C CNN
+F 2 "" H 3650 4900 50  0001 C CNN
+F 3 "" H 3650 4900 50  0001 C CNN
+	1    3650 4900
+	1    0    0    -1
+$EndComp
+Wire Wire Line
+	3650 4900 3650 4950
+Wire Wire Line
+	3650 5250 3650 5300
 Text Label 4450 3950 2    50   ~ 0
 I2C-SCL
@@
 P 6600 4750
 F 0 "BT701" H 6718 4846 50  0000 L CNN
-F 1 "Battery_Cell" H 6718 4755 50  0000 L CNN
+F 1 "RC2032" H 6718 4755 50  0000 L CNN
 F 2 "" V 6600 4810 50  0001 C CNN
 F 3 "~" V 6600 4810 50  0001 C CNN
@@
 AR Path="/5FD418B6" Ref="Y701"  Part="1"
 AR Path="/5FDBDABC/5FD418B6" Ref="Y701"  Part="1"
-F 0 "Y701" V 5105 5398 45  0000 L CNN
-F 1 "CRYSTAL-32.768KHZSMD-3.2X1.5" V 5189 5398 45  0000 L CNN
+F 0 "Y701" V 5100 5200 45  0000 R CNN
+F 1 "CRYSTAL-32.768KHZSMD-3.2X1.5" V 5200 5200 45  0000 R CNN
 F 2 "CRYSTAL-SMD-3.2X1.5MM" H 5200 5500 20  0001 C CNN
 F 3 "" H 5200 5300 50  0001 C CNN
-F 4 "XTAL-13062" V 5284 5398 60  0000 L CNN "Field4"
+F 4 "XTAL-13062" V 5300 5200 60  0000 R CNN "Field4"
 F 5 "-SLAVE" H 5200 5300 50  0001 C CNN "Config"
 	1    5200 5300
@@
 Wire Wire Line
 	3850 1000 3850 1250
+$Comp
+L Connector:TestPoint TP703
+U 1 1 5FE5017D
+P 6600 4400
+F 0 "TP703" H 6650 4500 50  0000 L CNN
+F 1 "RC2032" H 6658 4427 50  0001 L CNN
+F 2 "" H 6800 4400 50  0001 C CNN
+F 3 "~" H 6800 4400 50  0001 C CNN
+	1    6600 4400
+	1    0    0    -1
+$EndComp
+Wire Wire Line
+	6600 4400 6600 4450
+Connection ~ 6600 4450
 $EndSCHEMATC
