File: hardware/pcb/24-c-mechanics.sch (KiCad schematic (older format))
At the start: 7 parts, among them U301 VID28-05, U302 VID66-08, U303 AH3572, U304 AH3572

Commit message: Footprints (#2)
* Changed uC

* Updated processor pins and added testpoints

* Small changes

* Updated footprints

* changed crystals

* Created footprints and archived project

* Added motor footprint, made init pcb
Parts:
- added TP301: MA1, TestPoint:TestPoint_Pad_D2.0mm, symbol Connector:TestPoint
- added TP302: MA2, TestPoint:TestPoint_Pad_D2.0mm, symbol Connector:TestPoint
- added TP303: M-Rst, TestPoint:TestPoint_Pad_D2.0mm, symbol Connector:TestPoint
- added TP304: MA3, TestPoint:TestPoint_Pad_D2.0mm, symbol Connector:TestPoint
- added TP305: M-A-CW, TestPoint:TestPoint_Pad_D2.0mm, symbol Connector:TestPoint
- added TP306: M-A-Step, TestPoint:TestPoint_Pad_D2.0mm, symbol Connector:TestPoint
- added TP307: MA4, TestPoint:TestPoint_Pad_D2.0mm, symbol Connector:TestPoint
- added TP308: M-B-CW, TestPoint:TestPoint_Pad_D2.0mm, symbol Connector:TestPoint
- added TP309: M-B-Step, TestPoint:TestPoint_Pad_D2.0mm, symbol Connector:TestPoint
- added TP310: MB1, TestPoint:TestPoint_Pad_D2.0mm, symbol Connector:TestPoint
- added TP311: MB2, TestPoint:TestPoint_Pad_D2.0mm, symbol Connector:TestPoint
- added TP312: MB3, TestPoint:TestPoint_Pad_D2.0mm, symbol Connector:TestPoint
- added TP313: MB4, TestPoint:TestPoint_Pad_D2.0mm, symbol Connector:TestPoint
- added TP314: HAL-A, TestPoint:TestPoint_Pad_D2.0mm, symbol Connector:TestPoint
- added TP315: HAL-B, TestPoint:TestPoint_Pad_D2.0mm, symbol Connector:TestPoint
- C301: footprint C0603 -> Capacitor_SMD:C_0603_1608Metric
- R301, R302: footprint R0603 -> Resistor_SMD:R_0603_1608Metric
- U301: footprint (none) -> mvl-footprints:vid_28_05; symbol 24-clocks:VID28-05 -> 24-clocks-rescue:VID28-05-24-clocks
- U302: footprint TSOP-20 -> Package_SO:SOP-16_4.4x10.4mm_P1.27mm; symbol 24-clocks:VID66-08 -> 24-clocks-rescue:VID66-08-24-clocks
Connections:
- wire segments 52 -> 62
Other:
- moved on the sheet: C301, R301, R302, U303, U304

Commit message: Included all 3D files
Parts:
- U303, U304: footprint Package_TO_SOT_SMD:SOT-23 -> mvl-footprints:SOT-23-UD
Changed lines of the file:
@@
 F 0 "U303" H 5670 5096 50  0000 R CNN
 F 1 "AH3572" H 5670 5005 50  0000 R CNN
-F 2 "Package_TO_SOT_SMD:SOT-23" H 5950 5050 50  0001 C CNN
+F 2 "mvl-footprints:SOT-23-UD" H 5950 5050 50  0001 C CNN
 F 3 "https://www.diodes.com/assets/Datasheets/AH3572.pdf" H 5950 5050 50  0001 C CNN
 F 4 "-MASTER" H 6000 5050 50  0001 C CNN "Config"
@@
 F 0 "U304" H 7870 5096 50  0000 R CNN
 F 1 "AH3572" H 7870 5005 50  0000 R CNN
-F 2 "Package_TO_SOT_SMD:SOT-23" H 8150 5050 50  0001 C CNN
+F 2 "mvl-footprints:SOT-23-UD" H 8150 5050 50  0001 C CNN
 F 3 "https://www.diodes.com/assets/Datasheets/AH3572.pdf" H 8150 5050 50  0001 C CNN
 F 4 "-MASTER" H 8200 5050 50  0001 C CNN "Config"

Commit message: Mixed changes
Parts:
- added U305, U306: AH3572, Package_TO_SOT_SMD:TSOT-23, symbol Sensor_Magnetic:SM351LT
Connections:
- net +3V3: now also U305.1 (VCC), U306.1 (VCC)
- net GND: now also U305.3 (GND), U306.3 (GND)
- net HAL-A: now also U305.2 (OUTPUT)
- net HAL-B: now also U306.2 (OUTPUT)
Other:
- moved on the sheet: C301, R301, R302, TP301, TP302, TP303, TP304, TP305, TP306, TP307, TP308, TP309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
