File: hardware/pcb/24-c-mechanics.sch (KiCad schematic (older format))
At the start: 8 parts

Commit message: Created variants
Parts:
- C301: renamed from C?; Config (none) -> -MASTER
- R301, R302: renamed from R?; Config (none) -> -MASTER
- U301, U302, U303, U304: renamed from U?; Config (none) -> -MASTER
Changed lines of the file:
@@
 EESchema Schematic File Version 4
-EELAYER 30 0
+LIBS:24-clocks-cache
+EELAYER 29 0
 EELAYER END
 $Descr A4 11693 8268
 encoding utf-8
-Sheet 2 7
+Sheet 3 7
 Title "24 Clocks"
 Date "2020-12-06"
@@
 P 6800 2300
 AR Path="/5FCE4F17" Ref="U?"  Part="1"
-AR Path="/5FCDA719/5FCE4F17" Ref="U?"  Part="1"
-F 0 "U?" H 6775 3165 50  0000 C CNN
+AR Path="/5FCDA719/5FCE4F17" Ref="U302"  Part="1"
+F 0 "U302" H 6775 3165 50  0000 C CNN
 F 1 "VID66-08" H 6775 3074 50  0000 C CNN
 F 2 "TSOP-20" H 6250 2000 50  0001 C CNN
 F 3 "" H 6250 2000 50  0001 C CNN
+F 4 "-MASTER" H 6800 2300 50  0001 C CNN "Config"
 	1    6800 2300
 	1    0    0    -1
@@
 P 8400 1750
 AR Path="/5FCE4F23" Ref="U?"  Part="1"
-AR Path="/5FCDA719/5FCE4F23" Ref="U?"  Part="1"
-F 0 "U?" H 8400 2115 50  0000 C CNN
+AR Path="/5FCDA719/5FCE4F23" Ref="U301"  Part="1"
+F 0 "U301" H 8400 2115 50  0000 C CNN
 F 1 "VID28-05" H 8400 2024 50  0000 C CNN
 F 2 "" H 8400 1400 50  0001 C CNN
 F 3 "" H 8050 1750 50  0001 C CNN
+F 4 "-MASTER" H 8400 1750 50  0001 C CNN "Config"
 	1    8400 1750
 	1    0    0    -1
@@
 P 8400 2500
 AR Path="/5FCE4F29" Ref="U?"  Part="2"
-AR Path="/5FCDA719/5FCE4F29" Ref="U?"  Part="2"
-F 0 "U?" H 8400 2865 50  0000 C CNN
+AR Path="/5FCDA719/5FCE4F29" Ref="U301"  Part="2"
+F 0 "U301" H 8400 2865 50  0000 C CNN
 F 1 "VID28-05" H 8400 2774 50  0000 C CNN
 F 2 "" H 8400 2150 50  0001 C CNN
 F 3 "" H 8050 2500 50  0001 C CNN
+F 4 "-MASTER" H 8400 2500 50  0001 C CNN "Config"
 	2    8400 2500
 	1    0    0    -1
@@
 P 5300 2400
 AR Path="/5FCE4F4F" Ref="#PWR?"  Part="1"
-AR Path="/5FCDA719/5FCE4F4F" Ref="#PWR?"  Part="1"
-F 0 "#PWR?" H 5300 2250 50  0001 C CNN
+AR Path="/5FCDA719/5FCE4F4F" Ref="#PWR0301"  Part="1"
+F 0 "#PWR0301" H 5300 2250 50  0001 C CNN
 F 1 "+5V" H 5315 2573 50  0000 C CNN
 F 2 "" H 5300 2400 50  0001 C CNN
@@
 P 5300 2950
 AR Path="/5FCE4F55" Ref="#PWR?"  Part="1"
-AR Path="/5FCDA719/5FCE4F55" Ref="#PWR?"  Part="1"
-F 0 "#PWR?" H 5300 2700 50  0001 C CNN
+AR Path="/5FCDA719/5FCE4F55" Ref="#PWR0302"  Part="1"
+F 0 "#PWR0302" H 5300 2700 50  0001 C CNN
 F 1 "GND" H 5305 2777 50  0000 C CNN
 F 2 "" H 5300 2950 50  0001 C CNN
@@
 P 6100 2750
 AR Path="/5FCE4F62" Ref="C?"  Part="1"
-AR Path="/5FCDA719/5FCE4F62" Ref="C?"  Part="1"
-F 0 "C?" H 5986 2704 50  0000 R CNN
+AR Path="/5FCDA719/5FCE4F62" Ref="C301"  Part="1"
+F 0 "C301" H 5986 2704 50  0000 R CNN
 F 1 "100nF" H 5986 2795 50  0000 R CNN
 F 2 "C0603" H 6138 2600 50  0001 C CNN
 F 3 "~" H 6100 2750 50  0001 C CNN
+F 4 "-MASTER" H 6100 2750 50  0001 C CNN "Config"
 	1    6100 2750
 	1    0    0    1
@@
 P 6350 5000
 AR Path="/5FCEC14D" Ref="U?"  Part="1"
-AR Path="/5FCDA719/5FCEC14D" Ref="U?"  Part="1"
-F 0 "U?" H 6020 5046 50  0000 R CNN
+AR Path="/5FCDA719/5FCEC14D" Ref="U303"  Part="1"
+F 0 "U303" H 6020 5046 50  0000 R CNN
 F 1 "AH3572" H 6020 4955 50  0000 R CNN
 F 2 "Package_TO_SOT_SMD:SOT-23" H 6300 5000 50  0001 C CNN
 F 3 "https://www.diodes.com/assets/Datasheets/AH3572.pdf" H 6300 5000 50  0001 C CNN
+F 4 "-MASTER" H 6350 5000 50  0001 C CNN "Config"
 	1    6350 5000
 	-1   0    0    -1
@@
 P 6550 4600
 AR Path="/5FCEC153" Ref="#PWR?"  Part="1"
-AR Path="/5FCDA719/5FCEC153" Ref="#PWR?"  Part="1"
-F 0 "#PWR?" H 6550 4450 50  0001 C CNN
+AR Path="/5FCDA719/5FCEC153" Ref="#PWR0304"  Part="1"
+F 0 "#PWR0304" H 6550 4450 50  0001 C CNN
 F 1 "+3V3" H 6565 4773 50  0000 C CNN
 F 2 "" H 6550 4600 50  0001 C CNN
@@
 P 5750 4600
 AR Path="/5FCEC159" Ref="#PWR?"  Part="1"
-AR Path="/5FCDA719/5FCEC159" Ref="#PWR?"  Part="1"
-F 0 "#PWR?" H 5750 4450 50  0001 C CNN
+AR Path="/5FCDA719/5FCEC159" Ref="#PWR0303"  Part="1"
+F 0 "#PWR0303" H 5750 4450 50  0001 C CNN
 F 1 "+3V3" H 5765 4773 50  0000 C CNN
 F 2 "" H 5750 4600 50  0001 C CNN
@@
 P 6550 5350
 AR Path="/5FCEC15F" Ref="#PWR?"  Part="1"
-AR Path="/5FCDA719/5FCEC15F" Ref="#PWR?"  Part="1"
-F 0 "#PWR?" H 6550 5100 50  0001 C CNN
+AR Path="/5FCDA719/5FCEC15F" Ref="#PWR0307"  Part="1"
+F 0 "#PWR0307" H 6550 5100 50  0001 C CNN
 F 1 "GND" H 6555 5177 50  0000 C CNN
 F 2 "" H 6550 5350 50  0001 C CNN
@@
 P 5750 4800
 AR Path="/5FCEC165" Ref="R?"  Part="1"
-AR Path="/5FCDA719/5FCEC165" Ref="R?"  Part="1"
-F 0 "R?" H 5820 4846 50  0000 L CNN
+AR Path="/5FCDA719/5FCEC165" Ref="R301"  Part="1"
+F 0 "R301" H 5820 4846 50  0000 L CNN
 F 1 "10k" H 5820 4755 50  0000 L CNN
 F 2 "R0603" V 5680 4800 50  0001 C CNN
 F 3 "~" H 5750 4800 50  0001 C CNN
+F 4 "-MASTER" H 5750 4800 50  0001 C CNN "Config"
 	1    5750 4800
 	1    0    0    -1
@@
 P 8550 5000
 AR Path="/5FCEC173" Ref="U?"  Part="1"
-AR Path="/5FCDA719/5FCEC173" Ref="U?"  Part="1"
-F 0 "U?" H 8220 5046 50  0000 R CNN
+AR Path="/5FCDA719/5FCEC173" Ref="U304"  Part="1"
+F 0 "U304" H 8220 5046 50  0000 R CNN
 F 1 "AH3572" H 8220 4955 50  0000 R CNN
 F 2 "Package_TO_SOT_SMD:SOT-23" H 8500 5000 50  0001 C CNN
 F 3 "https://www.diodes.com/assets/Datasheets/AH3572.pdf" H 8500 5000 50  0001 C CNN
+F 4 "-MASTER" H 8550 5000 50  0001 C CNN "Config"
 	1    8550 5000
 	-1   0    0    -1
@@
 P 8750 4600
 AR Path="/5FCEC179" Ref="#PWR?"  Part="1"
-AR Path="/5FCDA719/5FCEC179" Ref="#PWR?"  Part="1"
-F 0 "#PWR?" H 8750 4450 50  0001 C CNN
+AR Path="/5FCDA719/5FCEC179" Ref="#PWR0306"  Part="1"
+F 0 "#PWR0306" H 8750 4450 50  0001 C CNN
 F 1 "+3V3" H 8765 4773 50  0000 C CNN
 F 2 "" H 8750 4600 50  0001 C CNN
@@
 P 7950 4600
 AR Path="/5FCEC17F" Ref="#PWR?"  Part="1"
-AR Path="/5FCDA719/5FCEC17F" Ref="#PWR?"  Part="1"
-F 0 "#PWR?" H 7950 4450 50  0001 C CNN
+AR Path="/5FCDA719/5FCEC17F" Ref="#PWR0305"  Part="1"
+F 0 "#PWR0305" H 7950 4450 50  0001 C CNN
 F 1 "+3V3" H 7965 4773 50  0000 C CNN
 F 2 "" H 7950 4600 50  0001 C CNN
@@
 P 8750 5350
 AR Path="/5FCEC185" Ref="#PWR?"  Part="1"
-AR Path="/5FCDA719/5FCEC185" Ref="#PWR?"  Part="1"
-F 0 "#PWR?" H 8750 5100 50  0001 C CNN
+AR Path="/5FCDA719/5FCEC185" Ref="#PWR0308"  Part="1"
+F 0 "#PWR0308" H 8750 5100 50  0001 C CNN
 F 1 "GND" H 8755 5177 50  0000 C CNN
 F 2 "" H 8750 5350 50  0001 C CNN
@@
 P 7950 4800
 AR Path="/5FCEC18B" Ref="R?"  Part="1"
-AR Path="/5FCDA719/5FCEC18B" Ref="R?"  Part="1"
-F 0 "R?" H 8020 4846 50  0000 L CNN
+AR Path="/5FCDA719/5FCEC18B" Ref="R302"  Part="1"
+F 0 "R302" H 8020 4846 50  0000 L CNN
 F 1 "10k" H 8020 4755 50  0000 L CNN
 F 2 "R0603" V 7880 4800 50  0001 C CNN
 F 3 "~" H 7950 4800 50  0001 C CNN
+F 4 "-MASTER" H 7950 4800 50  0001 C CNN "Config"
 	1    7950 4800
 	1    0    0    -1

Commit message: Updated processor pins and added testpoints
Parts:
- added TP301: MA1, symbol Connector:TestPoint
- added TP302: MA2, symbol Connector:TestPoint
- added TP303: M-Rst, symbol Connector:TestPoint
- added TP304: MA3, symbol Connector:TestPoint
- added TP305: M-A-CW, symbol Connector:TestPoint
- added TP306: M-A-Step, symbol Connector:TestPoint
- added TP307: MA4, symbol Connector:TestPoint
- added TP308: M-B-CW, symbol Connector:TestPoint
- added TP309: M-B-Step, symbol Connector:TestPoint
- added TP310: MB1, symbol Connector:TestPoint
- added TP311: MB2, symbol Connector:TestPoint
- added TP312: MB3, symbol Connector:TestPoint
- added TP313: MB4, symbol Connector:TestPoint
- added TP314: HAL-A, symbol Connector:TestPoint
- added TP315: HAL-B, symbol Connector:TestPoint
Connections:
- wire segments 52 -> 62
Changed lines of the file:
@@
 	1    0    0    -1
 $EndComp
-Wire Wire Line
-	5500 1700 6200 1700
-Wire Wire Line
-	5500 1900 6200 1900
-Wire Wire Line
-	5500 2000 6200 2000
-Wire Wire Line
-	5500 2200 6200 2200
-Wire Wire Line
-	5500 2300 6200 2300
 Text Label 5500 2000 0    50   ~ 0
 M-A-Step
@@
 L power:+5V #PWR?
 U 1 1 5FCE4F4F
-P 5300 2400
+P 4850 2450
 AR Path="/5FCE4F4F" Ref="#PWR?"  Part="1"
 AR Path="/5FCDA719/5FCE4F4F" Ref="#PWR0301"  Part="1"
-F 0 "#PWR0301" H 5300 2250 50  0001 C CNN
-F 1 "+5V" H 5315 2573 50  0000 C CNN
-F 2 "" H 5300 2400 50  0001 C CNN
-F 3 "" H 5300 2400 50  0001 C CNN
-	1    5300 2400
+F 0 "#PWR0301" H 4850 2300 50  0001 C CNN
+F 1 "+5V" H 4865 2623 50  0000 C CNN
+F 2 "" H 4850 2450 50  0001 C CNN
+F 3 "" H 4850 2450 50  0001 C CNN
+	1    4850 2450
 	1    0    0    -1
 $EndComp
@@
 Wire Wire Line
 	5300 2900 6100 2900
-Wire Wire Line
-	5300 2400 5300 2500
-Wire Wire Line
-	5300 2600 6100 2600
-Wire Wire Line
-	5300 2500 6200 2500
-Connection ~ 5300 2500
-Wire Wire Line
-	5300 2500 5300 2600
 $Comp
 L Device:C C?
@@
 Wire Wire Line
 	6550 5350 6550 5300
-Wire Wire Line
-	5750 5000 5100 5000
 Connection ~ 5750 5000
 Text Label 5100 5000 0    50   ~ 0
@@
 Wire Wire Line
 	8750 5350 8750 5300
-Wire Wire Line
-	7950 5000 7300 5000
 Connection ~ 7950 5000
 Text Label 7300 5000 0    50   ~ 0
@@
 Text Label 3700 4350 2    50   ~ 0
 HAL-B
+$Comp
+L Connector:TestPoint TP314
+U 1 1 5FF9BCFD
+P 5000 4900
+F 0 "TP314" H 5058 4972 50  0000 L CNN
+F 1 "HAL-A" H 5058 4927 50  0001 L CNN
+F 2 "" H 5200 4900 50  0001 C CNN
+F 3 "~" H 5200 4900 50  0001 C CNN
+	1    5000 4900
+	1    0    0    -1
+$EndComp
+Wire Wire Line
+	5000 4900 5000 5000
+Wire Wire Line
+	5000 5000 5750 5000
+$Comp
+L Connector:TestPoint TP315
+U 1 1 5FF9DCA7
+P 7200 4900
+F 0 "TP315" H 7258 4972 50  0000 L CNN
+F 1 "HAL-B" H 7258 4927 50  0001 L CNN
+F 2 "" H 7400 4900 50  0001 C CNN
+F 3 "~" H 7400 4900 50  0001 C CNN
+	1    7200 4900
+	1    0    0    -1
+$EndComp
+Wire Wire Line
+	7200 4900 7200 5000
+Wire Wire Line
+	7200 5000 7950 5000
+$Comp
+L Connector:TestPoint TP301
+U 1 1 5FF9F67F
+P 10100 1450
+F 0 "TP301" V 10203 1522 50  0000 C CNN
+F 1 "MA1" H 10158 1477 50  0001 L CNN
+F 2 "" H 10300 1450 50  0001 C CNN
+F 3 "~" H 10300 1450 50  0001 C CNN
+	1    10100 1450
+	0    1    -1   0
+$EndComp
+$Comp
+L Connector:TestPoint TP302
+U 1 1 5FFA0591
+P 10100 1650
+F 0 "TP302" V 10203 1722 50  0000 C CNN
+F 1 "MA2" H 10158 1677 50  0001 L CNN
+F 2 "" H 10300 1650 50  0001 C CNN
+F 3 "~" H 10300 1650 50  0001 C CNN
+	1    10100 1650
+	0    1    -1   0
+$EndComp
+$Comp
+L Connector:TestPoint TP304
+U 1 1 5FFA0852
+P 10100 1850
+F 0 "TP304" V 10203 1922 50  0000 C CNN
+F 1 "MA3" H 10158 1877 50  0001 L CNN
+F 2 "" H 10300 1850 50  0001 C CNN
+F 3 "~" H 10300 1850 50  0001 C CNN
+	1    10100 1850
+	0    1    -1   0
+$EndComp
+$Comp
+L Connector:TestPoint TP307
+U 1 1 5FFA0AC7
+P 10100 2050
+F 0 "TP307" V 10203 2122 50  0000 C CNN
+F 1 "MA4" H 10158 2077 50  0001 L CNN
+F 2 "" H 10300 2050 50  0001 C CNN
+F 3 "~" H 10300 2050 50  0001 C CNN
+	1    10100 2050
+	0    1    -1   0
+$EndComp
+Wire Wire Line
+	10100 1450 9700 1450
+Wire Wire Line
+	10100 1650 9700 1650
+Wire Wire Line
+	10100 1850 9700 1850
+Wire Wire Line
+	10100 2050 9700 2050
+$Comp
+L Connector:TestPoint TP310
+U 1 1 5FFAB35D
+P 10100 2400
+F 0 "TP310" V 10203 2472 50  0000 C CNN
+F 1 "MB1" H 10158 2427 50  0001 L CNN
+F 2 "" H 10300 2400 50  0001 C CNN
+F 3 "~" H 10300 2400 50  0001 C CNN
+	1    10100 2400
+	0    1    -1   0
+$EndComp
+$Comp
+L Connector:TestPoint TP311
+U 1 1 5FFAB363
+P 10100 2600
+F 0 "TP311" V 10203 2672 50  0000 C CNN
+F 1 "MB2" H 10158 2627 50  0001 L CNN
+F 2 "" H 10300 2600 50  0001 C CNN
+F 3 "~" H 10300 2600 50  0001 C CNN
+	1    10100 2600
+	0    1    -1   0
+$EndComp
+$Comp
+L Connector:TestPoint TP312
+U 1 1 5FFAB369
+P 10100 2800
+F 0 "TP312" V 10203 2872 50  0000 C CNN
+F 1 "MB3" H 10158 2827 50  0001 L CNN
+F 2 "" H 10300 2800 50  0001 C CNN
+F 3 "~" H 10300 2800 50  0001 C CNN
+	1    10100 2800
+	0    1    -1   0
+$EndComp
+$Comp
+L Connector:TestPoint TP313
+U 1 1 5FFAB36F
+P 10100 3000
+F 0 "TP313" V 10203 3072 50  0000 C CNN
+F 1 "MB4" H 10158 3027 50  0001 L CNN
+F 2 "" H 10300 3000 50  0001 C CNN
+F 3 "~" H 10300 3000 50  0001 C CNN
+	1    10100 3000
+	0    1    -1   0
+$EndComp
+Wire Wire Line
+	10100 2400 9700 2400
+Wire Wire Line
+	10100 2600 9700 2600
+Wire Wire Line
+	10100 2800 9700 2800
+Wire Wire Line
+	10100 3000 9700 3000
+Text Label 9700 1450 0    50   ~ 0
+MA1
+Text Label 9700 1650 0    50   ~ 0
+MA2
+Text Label 9700 1850 0    50   ~ 0
+MA3
+Text Label 9700 2050 0    50   ~ 0
+MA4
+Text Label 9700 2400 0    50   ~ 0
+MB1
+Text Label 9700 2600 0    50   ~ 0
+MB2
+Text Label 9700 2800 0    50   ~ 0
+MB3
+Text Label 9700 3000 0    50   ~ 0
+MB4
+$Comp
+L Connector:TestPoint TP309
+U 1 1 5FFB453E
+P 5450 2300
+F 0 "TP309" V 5450 2500 50  0000 L CNN
+F 1 "M-B-Step" H 5508 2327 50  0001 L CNN
+F 2 "" H 5650 2300 50  0001 C CNN
+F 3 "~" H 5650 2300 50  0001 C CNN
+	1    5450 2300
+	0    -1   1    0
+$EndComp
+$Comp
+L Connector:TestPoint TP308
+U 1 1 5FFBD755
+P 5450 2200
+F 0 "TP308" V 5450 2400 50  0000 L CNN
+F 1 "M-B-CW" H 5508 2227 50  0001 L CNN
+F 2 "" H 5650 2200 50  0001 C CNN
+F 3 "~" H 5650 2200 50  0001 C CNN
+	1    5450 2200
+	0    -1   1    0
+$EndComp
+$Comp
+L Connector:TestPoint TP306
+U 1 1 5FFBD8F9
+P 5450 2000
+F 0 "TP306" V 5450 2200 50  0000 L CNN
+F 1 "M-A-Step" H 5508 2027 50  0001 L CNN
+F 2 "" H 5650 2000 50  0001 C CNN
+F 3 "~" H 5650 2000 50  0001 C CNN
+	1    5450 2000
+	0    -1   1    0
+$EndComp
+$Comp
+L Connector:TestPoint TP305
+U 1 1 5FFBDA8A
+P 5450 1900
+F 0 "TP305" V 5450 2100 50  0000 L CNN
+F 1 "M-A-CW" H 5508 1927 50  0001 L CNN
+F 2 "" H 5650 1900 50  0001 C CNN
+F 3 "~" H 5650 1900 50  0001 C CNN
+	1    5450 1900
+	0    -1   1    0
+$EndComp
+$Comp
+L Connector:TestPoint TP303
+U 1 1 5FFBDBE2
+P 5450 1700
+F 0 "TP303" V 5450 1900 50  0000 L CNN
+F 1 "M-Rst" H 5508 1727 50  0001 L CNN
+F 2 "" H 5650 1700 50  0001 C CNN
+F 3 "~" H 5650 1700 50  0001 C CNN
+	1    5450 1700
+	0    -1   1    0
+$EndComp
+Wire Wire Line
+	4850 2450 4850 2500
+Wire Wire Line
+	4850 2600 4850 2500
+Connection ~ 4850 2500
+Wire Wire Line
+	4850 2500 6200 2500
+Wire Wire Line
+	4850 2600 6100 2600
+Wire Wire Line
+	5450 2300 6200 2300
+Wire Wire Line
+	5450 2200 6200 2200
+Wire Wire Line
+	5450 2000 6200 2000
+Wire Wire Line
+	5450 1900 6200 1900
+Wire Wire Line
+	5450 1700 6200 1700
 $EndSCHEMATC

Commit message: Small changes
Other:
- moved on the sheet: C301, R301, R302, TP301, TP302, TP303, TP304, TP305, TP306, TP307, TP308, TP309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

Commit message: Updated footprints
Parts:
- C301: footprint C0603 -> Capacitor_SMD:C_0603_1608Metric
- R301, R302: footprint R0603 -> Resistor_SMD:R_0603_1608Metric
- TP301, TP302, TP303, TP304, TP305, TP306, TP307, TP308, TP309, TP310, TP311, TP312, TP313, TP314, TP315: footprint (none) -> TestPoint:TestPoint_Pad_1.5x1.5mm
- U302: footprint TSOP-20 -> Package_SO:SOP-16_4.4x10.4mm_P1.27mm
Changed lines of the file:
@@
 F 0 "U302" H 6425 3215 50  0000 C CNN
 F 1 "VID66-08" H 6425 3124 50  0000 C CNN
-F 2 "TSOP-20" H 5900 2050 50  0001 C CNN
+F 2 "Package_SO:SOP-16_4.4x10.4mm_P1.27mm" H 5900 2050 50  0001 C CNN
 F 3 "http://www.vidmotion.com.cn/UploadFile/down/2009111391710_VID6608%20manual%20060927.pdf" H 5900 2050 50  0001 C CNN
 F 4 "-MASTER" H 6450 2350 50  0001 C CNN "Config"
@@
 F 0 "C301" H 5636 2754 50  0000 R CNN
 F 1 "100nF" H 5636 2845 50  0000 R CNN
-F 2 "C0603" H 5788 2650 50  0001 C CNN
+F 2 "Capacitor_SMD:C_0603_1608Metric" H 5788 2650 50  0001 C CNN
 F 3 "~" H 5750 2800 50  0001 C CNN
 F 4 "-MASTER" H 5750 2800 50  0001 C CNN "Config"
@@
 F 0 "R301" H 5470 4896 50  0000 L CNN
 F 1 "10k" H 5470 4805 50  0000 L CNN
-F 2 "R0603" V 5330 4850 50  0001 C CNN
+F 2 "Resistor_SMD:R_0603_1608Metric" V 5330 4850 50  0001 C CNN
 F 3 "~" H 5400 4850 50  0001 C CNN
 F 4 "-MASTER" H 5400 4850 50  0001 C CNN "Config"
@@
 F 0 "R302" H 7670 4896 50  0000 L CNN
 F 1 "10k" H 7670 4805 50  0000 L CNN
-F 2 "R0603" V 7530 4850 50  0001 C CNN
+F 2 "Resistor_SMD:R_0603_1608Metric" V 7530 4850 50  0001 C CNN
 F 3 "~" H 7600 4850 50  0001 C CNN
 F 4 "-MASTER" H 7600 4850 50  0001 C CNN "Config"
@@
 F 0 "TP314" H 4708 5022 50  0000 L CNN
 F 1 "HAL-A" H 4708 4977 50  0001 L CNN
-F 2 "" H 4850 4950 50  0001 C CNN
+F 2 "TestPoint:TestPoint_Pad_1.5x1.5mm" H 4850 4950 50  0001 C CNN
 F 3 "~" H 4850 4950 50  0001 C CNN
 	1    4650 4950
@@
 F 0 "TP315" H 6908 5022 50  0000 L CNN
 F 1 "HAL-B" H 6908 4977 50  0001 L CNN
-F 2 "" H 7050 4950 50  0001 C CNN
+F 2 "TestPoint:TestPoint_Pad_1.5x1.5mm" H 7050 4950 50  0001 C CNN
 F 3 "~" H 7050 4950 50  0001 C CNN
 	1    6850 4950
@@
 F 0 "TP301" V 9350 2000 50  0000 L CNN
 F 1 "MA1" H 9408 1827 50  0001 L CNN
-F 2 "" H 9550 1800 50  0001 C CNN
+F 2 "TestPoint:TestPoint_Pad_1.5x1.5mm" H 9550 1800 50  0001 C CNN
 F 3 "~" H 9550 1800 50  0001 C CNN
 	1    9350 1800
@@
 F 0 "TP302" V 9350 2100 50  0000 L CNN
 F 1 "MA2" H 9408 1927 50  0001 L CNN
-F 2 "" H 9550 1900 50  0001 C CNN
+F 2 "TestPoint:TestPoint_Pad_1.5x1.5mm" H 9550 1900 50  0001 C CNN
 F 3 "~" H 9550 1900 50  0001 C CNN
 	1    9350 1900
@@
 F 0 "TP304" V 9350 2200 50  0000 L CNN
 F 1 "MA3" H 9408 2027 50  0001 L CNN
-F 2 "" H 9550 2000 50  0001 C CNN
+F 2 "TestPoint:TestPoint_Pad_1.5x1.5mm" H 9550 2000 50  0001 C CNN
 F 3 "~" H 9550 2000 50  0001 C CNN
 	1    9350 2000
@@
 F 0 "TP307" V 9350 2300 50  0000 L CNN
 F 1 "MA4" H 9408 2127 50  0001 L CNN
-F 2 "" H 9550 2100 50  0001 C CNN
+F 2 "TestPoint:TestPoint_Pad_1.5x1.5mm" H 9550 2100 50  0001 C CNN
 F 3 "~" H 9550 2100 50  0001 C CNN
 	1    9350 2100
@@
 F 0 "TP310" V 9350 2750 50  0000 L CNN
 F 1 "MB1" H 9408 2577 50  0001 L CNN
-F 2 "" H 9550 2550 50  0001 C CNN
+F 2 "TestPoint:TestPoint_Pad_1.5x1.5mm" H 9550 2550 50  0001 C CNN
 F 3 "~" H 9550 2550 50  0001 C CNN
 	1    9350 2550
@@
 F 0 "TP311" V 9350 2850 50  0000 L CNN
 F 1 "MB2" H 9408 2677 50  0001 L CNN
-F 2 "" H 9550 2650 50  0001 C CNN
+F 2 "TestPoint:TestPoint_Pad_1.5x1.5mm" H 9550 2650 50  0001 C CNN
 F 3 "~" H 9550 2650 50  0001 C CNN
 	1    9350 2650
@@
 F 0 "TP312" V 9350 2950 50  0000 L CNN
 F 1 "MB3" H 9408 2777 50  0001 L CNN
-F 2 "" H 9550 2750 50  0001 C CNN
+F 2 "TestPoint:TestPoint_Pad_1.5x1.5mm" H 9550 2750 50  0001 C CNN
 F 3 "~" H 9550 2750 50  0001 C CNN
 	1    9350 2750
@@
 F 0 "TP313" V 9350 3050 50  0000 L CNN
 F 1 "MB4" H 9408 2877 50  0001 L CNN
-F 2 "" H 9550 2850 50  0001 C CNN
+F 2 "TestPoint:TestPoint_Pad_1.5x1.5mm" H 9550 2850 50  0001 C CNN
 F 3 "~" H 9550 2850 50  0001 C CNN
 	1    9350 2850
@@
 F 0 "TP309" V 5100 2550 50  0000 L CNN
 F 1 "M-B-Step" H 5158 2377 50  0001 L CNN
-F 2 "" H 5300 2350 50  0001 C CNN
+F 2 "TestPoint:TestPoint_Pad_1.5x1.5mm" H 5300 2350 50  0001 C CNN
 F 3 "~" H 5300 2350 50  0001 C CNN
 	1    5100 2350
@@
 F 0 "TP308" V 5100 2450 50  0000 L CNN
 F 1 "M-B-CW" H 5158 2277 50  0001 L CNN
-F 2 "" H 5300 2250 50  0001 C CNN
+F 2 "TestPoint:TestPoint_Pad_1.5x1.5mm" H 5300 2250 50  0001 C CNN
 F 3 "~" H 5300 2250 50  0001 C CNN
 	1    5100 2250
@@
 F 0 "TP306" V 5100 2250 50  0000 L CNN
 F 1 "M-A-Step" H 5158 2077 50  0001 L CNN
-F 2 "" H 5300 2050 50  0001 C CNN
+F 2 "TestPoint:TestPoint_Pad_1.5x1.5mm" H 5300 2050 50  0001 C CNN
 F 3 "~" H 5300 2050 50  0001 C CNN
 	1    5100 2050
@@
 F 0 "TP305" V 5100 2150 50  0000 L CNN
 F 1 "M-A-CW" H 5158 1977 50  0001 L CNN
-F 2 "" H 5300 1950 50  0001 C CNN
+F 2 "TestPoint:TestPoint_Pad_1.5x1.5mm" H 5300 1950 50  0001 C CNN
 F 3 "~" H 5300 1950 50  0001 C CNN
 	1    5100 1950
@@
 F 0 "TP303" V 5100 1950 50  0000 L CNN
 F 1 "M-Rst" H 5158 1777 50  0001 L CNN
-F 2 "" H 5300 1750 50  0001 C CNN
+F 2 "TestPoint:TestPoint_Pad_1.5x1.5mm" H 5300 1750 50  0001 C CNN
 F 3 "~" H 5300 1750 50  0001 C CNN
 	1    5100 1750

Commit message: Created footprints and archived project
Parts:
- U301: footprint (none) -> mvl-footprints:vid_28_05
Changed lines of the file:
@@
 F 0 "U301" H 8050 2165 50  0000 C CNN
 F 1 "VID28-05" H 8050 2074 50  0000 C CNN
-F 2 "" H 8050 1450 50  0001 C CNN
+F 2 "mvl-footprints:vid_28_05" H 8050 1450 50  0001 C CNN
 F 3 "" H 7700 1800 50  0001 C CNN
 F 4 "-MASTER" H 8050 1800 50  0001 C CNN "Config"
@@
 F 0 "U301" H 8050 2915 50  0000 C CNN
 F 1 "VID28-05" H 8050 2824 50  0000 C CNN
-F 2 "" H 8050 2200 50  0001 C CNN
+F 2 "mvl-footprints:vid_28_05" H 8050 2200 50  0001 C CNN
 F 3 "" H 7700 2550 50  0001 C CNN
 F 4 "-MASTER" H 8050 2550 50  0001 C CNN "Config"
