File: hardware/pcb/24-c-mechanics.sch (KiCad schematic (older format))
At the start: 22 parts, among them U301 VID28-05, U302 VID66-08, U303 AH3572, U304 AH3572

Commit message: Added motor footprint, made init pcb
Parts:
- TP301, TP302, TP303, TP304, TP305, TP306, TP307, TP308, TP309, TP310, TP311, TP312, TP313, TP314, TP315: footprint TestPoint:TestPoint_Pad_1.5x1.5mm -> TestPoint:TestPoint_Pad_D2.0mm
- U301: symbol 24-clocks:VID28-05 -> 24-clocks-rescue:VID28-05-24-clocks
- U302: symbol 24-clocks:VID66-08 -> 24-clocks-rescue:VID66-08-24-clocks
Changed lines of the file:
@@
 $EndDescr
 $Comp
-L 24-clocks:VID66-08 U?
+L 24-clocks-rescue:VID66-08-24-clocks U?
 U 1 1 5FCE4F17
 P 6450 2350
@@
 M-A-Step
 $Comp
-L 24-clocks:VID28-05 U?
+L 24-clocks-rescue:VID28-05-24-clocks U?
 U 1 1 5FCE4F23
 P 8050 1800
@@
 $EndComp
 $Comp
-L 24-clocks:VID28-05 U?
+L 24-clocks-rescue:VID28-05-24-clocks U?
 U 2 1 5FCE4F29
 P 8050 2550
@@
 F 0 "TP314" H 4708 5022 50  0000 L CNN
 F 1 "HAL-A" H 4708 4977 50  0001 L CNN
-F 2 "TestPoint:TestPoint_Pad_1.5x1.5mm" H 4850 4950 50  0001 C CNN
+F 2 "TestPoint:TestPoint_Pad_D2.0mm" H 4850 4950 50  0001 C CNN
 F 3 "~" H 4850 4950 50  0001 C CNN
 	1    4650 4950
@@
 F 0 "TP315" H 6908 5022 50  0000 L CNN
 F 1 "HAL-B" H 6908 4977 50  0001 L CNN
-F 2 "TestPoint:TestPoint_Pad_1.5x1.5mm" H 7050 4950 50  0001 C CNN
+F 2 "TestPoint:TestPoint_Pad_D2.0mm" H 7050 4950 50  0001 C CNN
 F 3 "~" H 7050 4950 50  0001 C CNN
 	1    6850 4950
@@
 F 0 "TP301" V 9350 2000 50  0000 L CNN
 F 1 "MA1" H 9408 1827 50  0001 L CNN
-F 2 "TestPoint:TestPoint_Pad_1.5x1.5mm" H 9550 1800 50  0001 C CNN
+F 2 "TestPoint:TestPoint_Pad_D2.0mm" H 9550 1800 50  0001 C CNN
 F 3 "~" H 9550 1800 50  0001 C CNN
 	1    9350 1800
@@
 F 0 "TP302" V 9350 2100 50  0000 L CNN
 F 1 "MA2" H 9408 1927 50  0001 L CNN
-F 2 "TestPoint:TestPoint_Pad_1.5x1.5mm" H 9550 1900 50  0001 C CNN
+F 2 "TestPoint:TestPoint_Pad_D2.0mm" H 9550 1900 50  0001 C CNN
 F 3 "~" H 9550 1900 50  0001 C CNN
 	1    9350 1900
@@
 F 0 "TP304" V 9350 2200 50  0000 L CNN
 F 1 "MA3" H 9408 2027 50  0001 L CNN
-F 2 "TestPoint:TestPoint_Pad_1.5x1.5mm" H 9550 2000 50  0001 C CNN
+F 2 "TestPoint:TestPoint_Pad_D2.0mm" H 9550 2000 50  0001 C CNN
 F 3 "~" H 9550 2000 50  0001 C CNN
 	1    9350 2000
@@
 F 0 "TP307" V 9350 2300 50  0000 L CNN
 F 1 "MA4" H 9408 2127 50  0001 L CNN
-F 2 "TestPoint:TestPoint_Pad_1.5x1.5mm" H 9550 2100 50  0001 C CNN
+F 2 "TestPoint:TestPoint_Pad_D2.0mm" H 9550 2100 50  0001 C CNN
 F 3 "~" H 9550 2100 50  0001 C CNN
 	1    9350 2100
@@
 F 0 "TP310" V 9350 2750 50  0000 L CNN
 F 1 "MB1" H 9408 2577 50  0001 L CNN
-F 2 "TestPoint:TestPoint_Pad_1.5x1.5mm" H 9550 2550 50  0001 C CNN
+F 2 "TestPoint:TestPoint_Pad_D2.0mm" H 9550 2550 50  0001 C CNN
 F 3 "~" H 9550 2550 50  0001 C CNN
 	1    9350 2550
@@
 F 0 "TP311" V 9350 2850 50  0000 L CNN
 F 1 "MB2" H 9408 2677 50  0001 L CNN
-F 2 "TestPoint:TestPoint_Pad_1.5x1.5mm" H 9550 2650 50  0001 C CNN
+F 2 "TestPoint:TestPoint_Pad_D2.0mm" H 9550 2650 50  0001 C CNN
 F 3 "~" H 9550 2650 50  0001 C CNN
 	1    9350 2650
@@
 F 0 "TP312" V 9350 2950 50  0000 L CNN
 F 1 "MB3" H 9408 2777 50  0001 L CNN
-F 2 "TestPoint:TestPoint_Pad_1.5x1.5mm" H 9550 2750 50  0001 C CNN
+F 2 "TestPoint:TestPoint_Pad_D2.0mm" H 9550 2750 50  0001 C CNN
 F 3 "~" H 9550 2750 50  0001 C CNN
 	1    9350 2750
@@
 F 0 "TP313" V 9350 3050 50  0000 L CNN
 F 1 "MB4" H 9408 2877 50  0001 L CNN
-F 2 "TestPoint:TestPoint_Pad_1.5x1.5mm" H 9550 2850 50  0001 C CNN
+F 2 "TestPoint:TestPoint_Pad_D2.0mm" H 9550 2850 50  0001 C CNN
 F 3 "~" H 9550 2850 50  0001 C CNN
 	1    9350 2850
@@
 F 0 "TP309" V 5100 2550 50  0000 L CNN
 F 1 "M-B-Step" H 5158 2377 50  0001 L CNN
-F 2 "TestPoint:TestPoint_Pad_1.5x1.5mm" H 5300 2350 50  0001 C CNN
+F 2 "TestPoint:TestPoint_Pad_D2.0mm" H 5300 2350 50  0001 C CNN
 F 3 "~" H 5300 2350 50  0001 C CNN
 	1    5100 2350
@@
 F 0 "TP308" V 5100 2450 50  0000 L CNN
 F 1 "M-B-CW" H 5158 2277 50  0001 L CNN
-F 2 "TestPoint:TestPoint_Pad_1.5x1.5mm" H 5300 2250 50  0001 C CNN
+F 2 "TestPoint:TestPoint_Pad_D2.0mm" H 5300 2250 50  0001 C CNN
 F 3 "~" H 5300 2250 50  0001 C CNN
 	1    5100 2250
@@
 F 0 "TP306" V 5100 2250 50  0000 L CNN
 F 1 "M-A-Step" H 5158 2077 50  0001 L CNN
-F 2 "TestPoint:TestPoint_Pad_1.5x1.5mm" H 5300 2050 50  0001 C CNN
+F 2 "TestPoint:TestPoint_Pad_D2.0mm" H 5300 2050 50  0001 C CNN
 F 3 "~" H 5300 2050 50  0001 C CNN
 	1    5100 2050
@@
 F 0 "TP305" V 5100 2150 50  0000 L CNN
 F 1 "M-A-CW" H 5158 1977 50  0001 L CNN
-F 2 "TestPoint:TestPoint_Pad_1.5x1.5mm" H 5300 1950 50  0001 C CNN
+F 2 "TestPoint:TestPoint_Pad_D2.0mm" H 5300 1950 50  0001 C CNN
 F 3 "~" H 5300 1950 50  0001 C CNN
 	1    5100 1950
@@
 F 0 "TP303" V 5100 1950 50  0000 L CNN
 F 1 "M-Rst" H 5158 1777 50  0001 L CNN
-F 2 "TestPoint:TestPoint_Pad_1.5x1.5mm" H 5300 1750 50  0001 C CNN
+F 2 "TestPoint:TestPoint_Pad_D2.0mm" H 5300 1750 50  0001 C CNN
 F 3 "~" H 5300 1750 50  0001 C CNN
 	1    5100 1750

Commit message: Finished PCB (#3)
* Created PCB outline and first placement

* Changed connectors

* Minor

* Included all 3D files

* Mixed changes

* Changed supply to 7V

* Archived PCB project

* Update 24-clocks-rescue.lib

* First placement

* Routed supplies

* Update 24-clocks.kicad_pcb

* Added routing

* Routed more nets

* Finished routing

* Archived project

* Replace hash and date

* minor

* Update pcb.yml

* Update pcb.yml

* Update pcb.yml

* Update pcb.yml

* Auto update commit date and hash

* Update output

* changed outputs

* Added layer to output

* Update hash and date also in sch

* Added caps to hall sensors

* Cleanup files
Parts:
- removed TP301: MA1, TestPoint:TestPoint_Pad_D2.0mm, symbol Connector:TestPoint
- removed TP302: MA2, TestPoint:TestPoint_Pad_D2.0mm, symbol Connector:TestPoint
- removed TP304: MA3, TestPoint:TestPoint_Pad_D2.0mm, symbol Connector:TestPoint
- removed TP307: MA4, TestPoint:TestPoint_Pad_D2.0mm, symbol Connector:TestPoint
- removed TP310: MB1, TestPoint:TestPoint_Pad_D2.0mm, symbol Connector:TestPoint
- removed TP311: MB2, TestPoint:TestPoint_Pad_D2.0mm, symbol Connector:TestPoint
- removed TP312: MB3, TestPoint:TestPoint_Pad_D2.0mm, symbol Connector:TestPoint
- removed TP313: MB4, TestPoint:TestPoint_Pad_D2.0mm, symbol Connector:TestPoint
- added C302, C303, C304, C305: 100nF, Capacitor_SMD:C_0603_1608Metric, symbol Device:C
- added U305, U306: AH3572, Package_TO_SOT_SMD:TSOT-23, symbol Sensor_Magnetic:SM351LT
- U301: footprint mvl-footprints:vid_28_05 -> mvl-footprints:BK30D-R5
- U303, U304: footprint Package_TO_SOT_SMD:SOT-23 -> mvl-footprints:SOT-23-UD; Config -MASTER -> -MASTER,-SLAVE
Connections:
- net +3V3: now also C302.2, C303.2, C304.2, C305.2, U305.1 (VCC), U306.1 (VCC)
- net GND: now also C302.1, C303.1, C304.1, C305.1, U305.3 (GND), U306.3 (GND)
- net HAL-A: now also U305.2 (OUTPUT)
- net HAL-B: now also U306.2 (OUTPUT)
Other:
- moved on the sheet: C301, R301, R302, TP303, TP305, TP306, TP308, TP309, TP314, TP315, U301A, U301B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
