File: hardware/pcb/24-c-uc.sch (KiCad schematic (older format))
At the start: 9 parts, among them J201 ST-LINK, J202 Debug UART, U201 STM32L151C8T6

Commit message: Footprints (#2)
* Changed uC

* Updated processor pins and added testpoints

* Small changes

* Updated footprints

* changed crystals

* Created footprints and archived project

* Added motor footprint, made init pcb
Parts:
- removed U201: STM32L151C8T6, Package_QFP:LQFP-48_7x7mm_P0.5mm, symbol MCU_ST_STM32L1:STM32L151C8Tx
- added C205, C206: 20pF, Capacitor_SMD:C_0603_1608Metric, symbol Device:C
- added JP203: Jumper_NO_Small, Jumper:SolderJumper-2_P1.3mm_Open_RoundedPad1.0x1.5mm, symbol Device:Jumper_NO_Small
- added R201: 4k7, Resistor_SMD:R_0603_1608Metric, symbol Device:R
- added R202, R203, R204, R205: 10k, Resistor_SMD:R_0603_1608Metric, symbol Device:R
- added TP201: SWO, TestPoint:TestPoint_Pad_D2.0mm, symbol Connector:TestPoint
- added TP202: uC-Rst, TestPoint:TestPoint_Pad_D2.0mm, symbol Connector:TestPoint
- added TP203: SWDCLK, TestPoint:TestPoint_Pad_D2.0mm, symbol Connector:TestPoint
- added TP204: SWDIO, TestPoint:TestPoint_Pad_D2.0mm, symbol Connector:TestPoint
- added TP205: 3V3, TestPoint:TestPoint_Pad_D2.0mm, symbol Connector:TestPoint
- added TP206: GND, TestPoint:TestPoint_Pad_D2.0mm, symbol Connector:TestPoint
- added TP207: BOOT0, TestPoint:TestPoint_Pad_D2.0mm, symbol Connector:TestPoint
- added TP208: BOOT1, TestPoint:TestPoint_Pad_D2.0mm, symbol Connector:TestPoint
- added TP209: uC-Debug-Rx, TestPoint:TestPoint_Pad_D2.0mm, symbol Connector:TestPoint
- added TP210: uC-Debug-Tx, TestPoint:TestPoint_Pad_D2.0mm, symbol Connector:TestPoint
- added TP211: HW-Version, TestPoint:TestPoint_Pad_D2.0mm, symbol Connector:TestPoint
- added U201: STM32F103C8Tx, Package_QFP:LQFP-48_7x7mm_P0.5mm, symbol MCU_ST_STM32F1:STM32F103C8Tx
- added Y201: 8MHz, Crystal:Crystal_SMD_5032-4Pin_5.0x3.2mm, symbol Device:Crystal_GND23_Small
- C201, C202, C203, C204: footprint C0603 -> Capacitor_SMD:C_0603_1608Metric
- J201: footprint (none) -> Connector_PinHeader_2.54mm:PinHeader_2x04_P2.54mm_Vertical
- J202: footprint (none) -> Connector_PinHeader_2.54mm:PinHeader_1x06_P2.54mm_Vertical
- JP201: footprint (none) -> Jumper:SolderJumper-2_P1.3mm_Bridged_RoundedPad1.0x1.5mm
- JP202: footprint (none) -> Jumper:SolderJumper-2_P1.3mm_Open_RoundedPad1.0x1.5mm
Connections:
- net labels added: BOOT1, HW-Version, SWO
- net labels removed: SWCLK, SWIM
- wire segments 90 -> 137
- no-connect marks 0 -> 16
Other:
- note added: "Hardware version"
- moved on the sheet: C201, C202, C203, C204, J202, JP202

Commit message: Included all 3D files
Parts:
- Y201: footprint Crystal:Crystal_SMD_5032-4Pin_5.0x3.2mm -> Crystal:Crystal_SMD_3225-4Pin_3.2x2.5mm
Changed lines of the file:
@@
 F 0 "Y201" V 3954 2494 50  0000 L CNN
 F 1 "8MHz" V 4045 2494 50  0000 L CNN
-F 2 "Crystal:Crystal_SMD_5032-4Pin_5.0x3.2mm" H 4000 2350 50  0001 C CNN
+F 2 "Crystal:Crystal_SMD_3225-4Pin_3.2x2.5mm" H 4000 2350 50  0001 C CNN
 F 3 "~" H 4000 2350 50  0001 C CNN
 	1    4000 2350

Commit message: Mixed changes
Parts:
- Y201: value 8MHz -> NX3225GD 8MHz; footprint Crystal:Crystal_SMD_3225-4Pin_3.2x2.5mm -> mvl-footprints:Crystal_SMD_3225-2Pin_3.2x2.5mm; symbol Device:Crystal_GND23_Small -> Device:Crystal_Small
Connections:
- net GND: no longer Y201.2, Y201.3
- net at C206.1, U201.6 (PD1): now also Y201.2; no longer Y201.4
Changed lines of the file:
@@
 	3650 2150 3600 2150
 Wire Wire Line
-	3600 2150 3600 2350
-Wire Wire Line
 	3600 2550 3650 2550
 Wire Wire Line
 	3950 2550 4000 2550
 Wire Wire Line
-	4600 2550 4600 2400
-Wire Wire Line
-	4600 2400 5000 2400
-Wire Wire Line
-	5000 2300 4600 2300
-Wire Wire Line
-	4600 2300 4600 2150
-Wire Wire Line
-	4600 2150 4000 2150
+	4750 2550 4750 2400
+Wire Wire Line
+	4750 2400 5000 2400
+Wire Wire Line
+	5000 2300 4750 2300
+Wire Wire Line
+	4750 2300 4750 2150
+Wire Wire Line
+	4750 2150 4000 2150
 Connection ~ 4000 2150
 Wire Wire Line
@@
 Connection ~ 4000 2550
 Wire Wire Line
-	4000 2550 4600 2550
+	4000 2550 4750 2550
 $Comp
 L power:GND #PWR?
@@
 	1400 6600 2100 6600
 $Comp
-L Device:Crystal_GND23_Small Y201
+L Device:Crystal_Small Y201
 U 1 1 5FE749A7
 P 4000 2350
-F 0 "Y201" V 3954 2494 50  0000 L CNN
-F 1 "8MHz" V 4045 2494 50  0000 L CNN
-F 2 "Crystal:Crystal_SMD_3225-4Pin_3.2x2.5mm" H 4000 2350 50  0001 C CNN
-F 3 "~" H 4000 2350 50  0001 C CNN
+F 0 "Y201" V 3950 2450 50  0000 L CNN
+F 1 "NX3225GD 8MHz" V 4050 2450 50  0000 L CNN
+F 2 "mvl-footprints:Crystal_SMD_3225-2Pin_3.2x2.5mm" H 4000 2350 50  0001 C CNN
+F 3 "https://www.ndk.com/images/products/catalog/c_NX3225GD_e.pdf" H 4000 2350 50  0001 C CNN
 	1    4000 2350
 	0    1    1    0
@@
 	4000 2450 4000 2550
 Wire Wire Line
-	3900 2350 3600 2350
-Connection ~ 3600 2350
-Wire Wire Line
-	3600 2350 3600 2550
-$Comp
-L power:GND #PWR?
-U 1 1 5FE85E24
-P 4100 2600
-AR Path="/5FE85E24" Ref="#PWR?"  Part="1"
-AR Path="/5FDEAABE/5FE85E24" Ref="#PWR0108"  Part="1"
-F 0 "#PWR0108" H 4100 2350 50  0001 C CNN
-F 1 "GND" H 4105 2427 50  0000 C CNN
-F 2 "" H 4100 2600 50  0001 C CNN
-F 3 "" H 4100 2600 50  0001 C CNN
-	1    4100 2600
-	1    0    0    -1
-$EndComp
-Wire Wire Line
-	4100 2600 4100 2350
+	3600 2150 3600 2550
 $EndSCHEMATC
