File: hardware/pcb/24-c-wifi.sch (KiCad schematic (older format))
At the start: 7 parts, among them J601 Conn_02x03_Odd_Even, U601 ESP32-WROOM-32D

Commit message: Footprints (#2)
* Changed uC

* Updated processor pins and added testpoints

* Small changes

* Updated footprints

* changed crystals

* Created footprints and archived project

* Added motor footprint, made init pcb
Parts:
- added TP601: uC-WiFi-Tx, TestPoint:TestPoint_Pad_D2.0mm, symbol Connector:TestPoint
- added TP602: uC-WiFi-Rx, TestPoint:TestPoint_Pad_D2.0mm, symbol Connector:TestPoint
- C601: footprint (none) -> Capacitor_SMD:C_Elec_10x10.2
- C602: footprint C0603 -> Capacitor_SMD:C_0603_1608Metric
- J601: footprint (none) -> Connector_PinHeader_1.27mm:PinHeader_2x03_P1.27mm_Vertical
- JP601: footprint (none) -> Jumper:SolderJumper-2_P1.3mm_Bridged_RoundedPad1.0x1.5mm
- R601, R602: footprint R0603 -> Resistor_SMD:R_0603_1608Metric
- U601: symbol 24-clocks:ESP32-WROOM-32D -> 24-clocks-rescue:ESP32-WROOM-32D-24-clocks
Connections:
- no-connect marks 0 -> 27
Changed lines of the file:
@@
 $EndDescr
 $Comp
-L 24-clocks:ESP32-WROOM-32D U?
+L 24-clocks-rescue:ESP32-WROOM-32D-24-clocks U?
 U 1 1 5FDA8E5C
 P 6000 4150
 AR Path="/5FDA8E5C" Ref="U?"  Part="1"
 AR Path="/5FDA43A0/5FDA8E5C" Ref="U601"  Part="1"
-F 0 "U601" H 5600 5550 50  0000 C CNN
+F 0 "U601" H 5700 5550 50  0000 C CNN
 F 1 "ESP32-WROOM-32D" H 6500 2750 50  0000 C CNN
 F 2 "RF_Module:ESP32-WROOM-32" H 6000 2650 50  0001 C CNN
@@
 F 0 "R601" H 5370 2796 50  0000 L CNN
 F 1 "10k" H 5370 2705 50  0000 L CNN
-F 2 "R0603" V 5230 2750 50  0001 C CNN
+F 2 "Resistor_SMD:R_0603_1608Metric" V 5230 2750 50  0001 C CNN
 F 3 "~" H 5300 2750 50  0001 C CNN
 F 4 "-SLAVE" H 5300 2750 50  0001 C CNN "Config"
@@
 F 0 "R602" H 6770 2796 50  0000 L CNN
 F 1 "10k" H 6770 2705 50  0000 L CNN
-F 2 "R0603" V 6630 2750 50  0001 C CNN
+F 2 "Resistor_SMD:R_0603_1608Metric" V 6630 2750 50  0001 C CNN
 F 3 "~" H 6700 2750 50  0001 C CNN
 F 4 "-SLAVE" H 6700 2750 50  0001 C CNN "Config"
@@
 Wire Wire Line
 	6600 3250 7150 3250
-Wire Wire Line
-	6600 3950 7150 3950
-Wire Wire Line
-	6600 4050 7150 4050
 Wire Wire Line
 	6700 2900 6700 2950
@@
 F 0 "C602" H 5715 1946 50  0000 L CNN
 F 1 "100nF" H 5715 1855 50  0000 L CNN
-F 2 "C0603" H 5638 1750 50  0001 C CNN
+F 2 "Capacitor_SMD:C_0603_1608Metric" H 5638 1750 50  0001 C CNN
 F 3 "~" H 5600 1900 50  0001 C CNN
 F 4 "-SLAVE" H 5600 1900 50  0001 C CNN "Config"
@@
 F 0 "C601" H 5268 1946 50  0000 L CNN
 F 1 "22uF" H 5268 1855 50  0000 L CNN
-F 2 "" H 5188 1750 50  0001 C CNN
+F 2 "Capacitor_SMD:C_Elec_10x10.2" H 5188 1750 50  0001 C CNN
 F 3 "~" H 5150 1900 50  0001 C CNN
 F 4 "-SLAVE" H 5150 1900 50  0001 C CNN "Config"
@@
 F 0 "J601" H 9000 2975 50  0000 C CNN
 F 1 "Conn_02x03_Odd_Even" H 9000 2976 50  0001 C CNN
-F 2 "" H 8950 2750 50  0001 C CNN
+F 2 "Connector_PinHeader_1.27mm:PinHeader_2x03_P1.27mm_Vertical" H 8950 2750 50  0001 C CNN
 F 3 "~" H 8950 2750 50  0001 C CNN
 F 4 "-SLAVE" H 8950 2750 50  0001 C CNN "Config"
@@
 F 0 "JP601" H 9500 2771 50  0000 C CNN
 F 1 "Jumper_NC_Small" H 9500 2771 50  0001 C CNN
-F 2 "" H 9500 2650 50  0001 C CNN
+F 2 "Jumper:SolderJumper-2_P1.3mm_Bridged_RoundedPad1.0x1.5mm" H 9500 2650 50  0001 C CNN
 F 3 "~" H 9500 2650 50  0001 C CNN
 	1    9500 2650
@@
 Text Label 2950 2500 2    50   ~ 0
 uC-WiFi-Rx
+NoConn ~ 6600 5250
+NoConn ~ 6600 5150
+NoConn ~ 6600 5050
+NoConn ~ 6600 4950
+NoConn ~ 6600 4850
+NoConn ~ 6600 4750
+NoConn ~ 6600 4650
+NoConn ~ 6600 4550
+NoConn ~ 6600 4450
+NoConn ~ 6600 4350
+NoConn ~ 6600 4250
+NoConn ~ 6600 4150
+NoConn ~ 6600 3850
+NoConn ~ 6600 3750
+NoConn ~ 6600 3650
+NoConn ~ 6600 3550
+NoConn ~ 6600 3450
+NoConn ~ 6600 3350
+NoConn ~ 6600 3150
+NoConn ~ 5400 4150
+NoConn ~ 5400 4250
+NoConn ~ 5400 4350
+NoConn ~ 5400 4450
+NoConn ~ 5400 4550
+NoConn ~ 5400 4650
+NoConn ~ 5400 3250
+NoConn ~ 5400 3150
+$Comp
+L Connector:TestPoint TP601
+U 1 1 5FE4BA8B
+P 7200 3950
+F 0 "TP601" V 7200 4138 50  0000 L CNN
+F 1 "uC-WiFi-Tx" V 7245 4138 50  0001 L CNN
+F 2 "TestPoint:TestPoint_Pad_D2.0mm" H 7400 3950 50  0001 C CNN
+F 3 "~" H 7400 3950 50  0001 C CNN
+	1    7200 3950
+	0    1    1    0
+$EndComp
+$Comp
+L Connector:TestPoint TP602
+U 1 1 5FE4C9AE
+P 7200 4050
+F 0 "TP602" V 7200 4238 50  0000 L CNN
+F 1 "uC-WiFi-Rx" V 7245 4238 50  0001 L CNN
+F 2 "TestPoint:TestPoint_Pad_D2.0mm" H 7400 4050 50  0001 C CNN
+F 3 "~" H 7400 4050 50  0001 C CNN
+	1    7200 4050
+	0    1    1    0
+$EndComp
+Wire Wire Line
+	6600 3950 7200 3950
+Wire Wire Line
+	6600 4050 7200 4050
 $EndSCHEMATC
