File: hardware/pcb/24-c-wifi.sch (KiCad schematic (older format))
At the start: 7 parts

Commit message: Created variants
Parts:
- C601, C602: renamed from C?; Config (none) -> -SLAVE
- J601: renamed from J?; Config (none) -> -SLAVE
- R601, R602: renamed from R?; Config (none) -> -SLAVE
- U601: renamed from U?; Config (none) -> -SLAVE
- gave numbers to parts that had none: 1
Changed lines of the file:
@@
 EESchema Schematic File Version 4
-EELAYER 30 0
+LIBS:24-clocks-cache
+EELAYER 29 0
 EELAYER END
 $Descr A4 11693 8268
 encoding utf-8
-Sheet 5 7
+Sheet 6 7
 Title "24 Clocks"
 Date "2020-12-06"
@@
 P 6000 4150
 AR Path="/5FDA8E5C" Ref="U?"  Part="1"
-AR Path="/5FDA43A0/5FDA8E5C" Ref="U?"  Part="1"
-F 0 "U?" H 5600 5550 50  0000 C CNN
+AR Path="/5FDA43A0/5FDA8E5C" Ref="U601"  Part="1"
+F 0 "U601" H 5600 5550 50  0000 C CNN
 F 1 "ESP32-WROOM-32D" H 6500 2750 50  0000 C CNN
 F 2 "RF_Module:ESP32-WROOM-32" H 6000 2650 50  0001 C CNN
 F 3 "" H 5700 4200 50  0001 C CNN
+F 4 "-SLAVE" H 6000 4150 50  0001 C CNN "Config"
 	1    6000 4150
 	1    0    0    -1
@@
 P 5300 2550
 AR Path="/5FDA8E62" Ref="#PWR?"  Part="1"
-AR Path="/5FDA43A0/5FDA8E62" Ref="#PWR?"  Part="1"
-F 0 "#PWR?" H 5300 2400 50  0001 C CNN
+AR Path="/5FDA43A0/5FDA8E62" Ref="#PWR0604"  Part="1"
+F 0 "#PWR0604" H 5300 2400 50  0001 C CNN
 F 1 "+3V3" H 5315 2723 50  0000 C CNN
 F 2 "" H 5300 2550 50  0001 C CNN
@@
 P 5300 2750
 AR Path="/5FDA8E68" Ref="R?"  Part="1"
-AR Path="/5FDA43A0/5FDA8E68" Ref="R?"  Part="1"
-F 0 "R?" H 5370 2796 50  0000 L CNN
+AR Path="/5FDA43A0/5FDA8E68" Ref="R601"  Part="1"
+F 0 "R601" H 5370 2796 50  0000 L CNN
 F 1 "10k" H 5370 2705 50  0000 L CNN
 F 2 "R0603" V 5230 2750 50  0001 C CNN
 F 3 "~" H 5300 2750 50  0001 C CNN
+F 4 "-SLAVE" H 5300 2750 50  0001 C CNN "Config"
 	1    5300 2750
 	1    0    0    -1
@@
 P 6700 2550
 AR Path="/5FDA8E74" Ref="#PWR?"  Part="1"
-AR Path="/5FDA43A0/5FDA8E74" Ref="#PWR?"  Part="1"
-F 0 "#PWR?" H 6700 2400 50  0001 C CNN
+AR Path="/5FDA43A0/5FDA8E74" Ref="#PWR0605"  Part="1"
+F 0 "#PWR0605" H 6700 2400 50  0001 C CNN
 F 1 "+3V3" H 6715 2723 50  0000 C CNN
 F 2 "" H 6700 2550 50  0001 C CNN
@@
 P 6700 2750
 AR Path="/5FDA8E7A" Ref="R?"  Part="1"
-AR Path="/5FDA43A0/5FDA8E7A" Ref="R?"  Part="1"
-F 0 "R?" H 6770 2796 50  0000 L CNN
+AR Path="/5FDA43A0/5FDA8E7A" Ref="R602"  Part="1"
+F 0 "R602" H 6770 2796 50  0000 L CNN
 F 1 "10k" H 6770 2705 50  0000 L CNN
 F 2 "R0603" V 6630 2750 50  0001 C CNN
 F 3 "~" H 6700 2750 50  0001 C CNN
+F 4 "-SLAVE" H 6700 2750 50  0001 C CNN "Config"
 	1    6700 2750
 	1    0    0    -1
@@
 P 4900 1650
 AR Path="/5FDA8E8C" Ref="#PWR?"  Part="1"
-AR Path="/5FDA43A0/5FDA8E8C" Ref="#PWR?"  Part="1"
-F 0 "#PWR?" H 4900 1500 50  0001 C CNN
+AR Path="/5FDA43A0/5FDA8E8C" Ref="#PWR0601"  Part="1"
+F 0 "#PWR0601" H 4900 1500 50  0001 C CNN
 F 1 "+3V3" H 4915 1823 50  0000 C CNN
 F 2 "" H 4900 1650 50  0001 C CNN
@@
 P 6000 5600
 AR Path="/5FDA8E92" Ref="#PWR?"  Part="1"
-AR Path="/5FDA43A0/5FDA8E92" Ref="#PWR?"  Part="1"
-F 0 "#PWR?" H 6000 5350 50  0001 C CNN
+AR Path="/5FDA43A0/5FDA8E92" Ref="#PWR0608"  Part="1"
+F 0 "#PWR0608" H 6000 5350 50  0001 C CNN
 F 1 "GND" H 6005 5427 50  0000 C CNN
 F 2 "" H 6000 5600 50  0001 C CNN
@@
 P 5600 1900
 AR Path="/5FDA8E99" Ref="C?"  Part="1"
-AR Path="/5FDA43A0/5FDA8E99" Ref="C?"  Part="1"
-F 0 "C?" H 5715 1946 50  0000 L CNN
+AR Path="/5FDA43A0/5FDA8E99" Ref="C602"  Part="1"
+F 0 "C602" H 5715 1946 50  0000 L CNN
 F 1 "100nF" H 5715 1855 50  0000 L CNN
 F 2 "C0603" H 5638 1750 50  0001 C CNN
 F 3 "~" H 5600 1900 50  0001 C CNN
+F 4 "-SLAVE" H 5600 1900 50  0001 C CNN "Config"
 	1    5600 1900
 	1    0    0    -1
@@
 P 5600 2100
 AR Path="/5FDA8E9F" Ref="#PWR?"  Part="1"
-AR Path="/5FDA43A0/5FDA8E9F" Ref="#PWR?"  Part="1"
-F 0 "#PWR?" H 5600 1850 50  0001 C CNN
+AR Path="/5FDA43A0/5FDA8E9F" Ref="#PWR0603"  Part="1"
+F 0 "#PWR0603" H 5600 1850 50  0001 C CNN
 F 1 "GND" H 5605 1927 50  0000 C CNN
 F 2 "" H 5600 2100 50  0001 C CNN
@@
 P 5150 2100
 AR Path="/5FDA8EA6" Ref="#PWR?"  Part="1"
-AR Path="/5FDA43A0/5FDA8EA6" Ref="#PWR?"  Part="1"
-F 0 "#PWR?" H 5150 1850 50  0001 C CNN
+AR Path="/5FDA43A0/5FDA8EA6" Ref="#PWR0602"  Part="1"
+F 0 "#PWR0602" H 5150 1850 50  0001 C CNN
 F 1 "GND" H 5155 1927 50  0000 C CNN
 F 2 "" H 5150 2100 50  0001 C CNN
@@
 P 5150 1900
 AR Path="/5FDA8EAC" Ref="C?"  Part="1"
-AR Path="/5FDA43A0/5FDA8EAC" Ref="C?"  Part="1"
-F 0 "C?" H 5268 1946 50  0000 L CNN
+AR Path="/5FDA43A0/5FDA8EAC" Ref="C601"  Part="1"
+F 0 "C601" H 5268 1946 50  0000 L CNN
 F 1 "22uF" H 5268 1855 50  0000 L CNN
 F 2 "" H 5188 1750 50  0001 C CNN
 F 3 "~" H 5150 1900 50  0001 C CNN
+F 4 "-SLAVE" H 5150 1900 50  0001 C CNN "Config"
 	1    5150 1900
 	1    0    0    -1
@@
 P 8950 2750
 AR Path="/5FDADE19" Ref="J?"  Part="1"
-AR Path="/5FDA43A0/5FDADE19" Ref="J?"  Part="1"
-F 0 "J?" H 9000 2975 50  0000 C CNN
+AR Path="/5FDA43A0/5FDADE19" Ref="J601"  Part="1"
+F 0 "J601" H 9000 2975 50  0000 C CNN
 F 1 "Conn_02x03_Odd_Even" H 9000 2976 50  0001 C CNN
 F 2 "" H 8950 2750 50  0001 C CNN
 F 3 "~" H 8950 2750 50  0001 C CNN
+F 4 "-SLAVE" H 8950 2750 50  0001 C CNN "Config"
 	1    8950 2750
 	1    0    0    -1
@@
 P 9700 2900
 AR Path="/5FDADE27" Ref="#PWR?"  Part="1"
-AR Path="/5FDA43A0/5FDADE27" Ref="#PWR?"  Part="1"
-F 0 "#PWR?" H 9700 2650 50  0001 C CNN
+AR Path="/5FDA43A0/5FDADE27" Ref="#PWR0607"  Part="1"
+F 0 "#PWR0607" H 9700 2650 50  0001 C CNN
 F 1 "GND" H 9705 2727 50  0000 C CNN
 F 2 "" H 9700 2900 50  0001 C CNN
@@
 P 9700 2600
 AR Path="/5FDADE2D" Ref="#PWR?"  Part="1"
-AR Path="/5FDA43A0/5FDADE2D" Ref="#PWR?"  Part="1"
-F 0 "#PWR?" H 9700 2450 50  0001 C CNN
+AR Path="/5FDA43A0/5FDADE2D" Ref="#PWR0606"  Part="1"
+F 0 "#PWR0606" H 9700 2450 50  0001 C CNN
 F 1 "+3V3" H 9715 2773 50  0000 C CNN
 F 2 "" H 9700 2600 50  0001 C CNN
@@
 P 9500 2650
 AR Path="/5FDADE37" Ref="JP?"  Part="1"
-AR Path="/5FDA43A0/5FDADE37" Ref="JP?"  Part="1"
-F 0 "JP?" H 9500 2771 50  0000 C CNN
+AR Path="/5FDA43A0/5FDADE37" Ref="JP601"  Part="1"
+F 0 "JP601" H 9500 2771 50  0000 C CNN
 F 1 "Jumper_NC_Small" H 9500 2771 50  0001 C CNN
 F 2 "" H 9500 2650 50  0001 C CNN

Commit message: Changed uC
Connections:
- no-connect marks 0 -> 27
Changed lines of the file:
@@
 EESchema Schematic File Version 4
-LIBS:24-clocks-cache
-EELAYER 29 0
+EELAYER 30 0
 EELAYER END
 $Descr A4 11693 8268
@@
 Text Label 2950 2500 2    50   ~ 0
 uC-WiFi-Rx
+NoConn ~ 6600 5250
+NoConn ~ 6600 5150
+NoConn ~ 6600 5050
+NoConn ~ 6600 4950
+NoConn ~ 6600 4850
+NoConn ~ 6600 4750
+NoConn ~ 6600 4650
+NoConn ~ 6600 4550
+NoConn ~ 6600 4450
+NoConn ~ 6600 4350
+NoConn ~ 6600 4250
+NoConn ~ 6600 4150
+NoConn ~ 6600 3850
+NoConn ~ 6600 3750
+NoConn ~ 6600 3650
+NoConn ~ 6600 3550
+NoConn ~ 6600 3450
+NoConn ~ 6600 3350
+NoConn ~ 6600 3150
+NoConn ~ 5400 4150
+NoConn ~ 5400 4250
+NoConn ~ 5400 4350
+NoConn ~ 5400 4450
+NoConn ~ 5400 4550
+NoConn ~ 5400 4650
+NoConn ~ 5400 3250
+NoConn ~ 5400 3150
 $EndSCHEMATC

Commit message: Small changes
Parts:
- added TP601: uC-WiFi-Tx, symbol Connector:TestPoint
- added TP602: uC-WiFi-Rx, symbol Connector:TestPoint
Changed lines of the file:
@@
 EESchema Schematic File Version 4
-EELAYER 30 0
+LIBS:24-clocks-cache
+EELAYER 29 0
 EELAYER END
 $Descr A4 11693 8268
@@
 AR Path="/5FDA8E5C" Ref="U?"  Part="1"
 AR Path="/5FDA43A0/5FDA8E5C" Ref="U601"  Part="1"
-F 0 "U601" H 5600 5550 50  0000 C CNN
+F 0 "U601" H 5700 5550 50  0000 C CNN
 F 1 "ESP32-WROOM-32D" H 6500 2750 50  0000 C CNN
 F 2 "RF_Module:ESP32-WROOM-32" H 6000 2650 50  0001 C CNN
@@
 Wire Wire Line
 	6600 3250 7150 3250
-Wire Wire Line
-	6600 3950 7150 3950
-Wire Wire Line
-	6600 4050 7150 4050
 Wire Wire Line
 	6700 2900 6700 2950
@@
 NoConn ~ 5400 3250
 NoConn ~ 5400 3150
+$Comp
+L Connector:TestPoint TP601
+U 1 1 5FE4BA8B
+P 7200 3950
+F 0 "TP601" V 7200 4138 50  0000 L CNN
+F 1 "uC-WiFi-Tx" V 7245 4138 50  0001 L CNN
+F 2 "" H 7400 3950 50  0001 C CNN
+F 3 "~" H 7400 3950 50  0001 C CNN
+	1    7200 3950
+	0    1    1    0
+$EndComp
+$Comp
+L Connector:TestPoint TP602
+U 1 1 5FE4C9AE
+P 7200 4050
+F 0 "TP602" V 7200 4238 50  0000 L CNN
+F 1 "uC-WiFi-Rx" V 7245 4238 50  0001 L CNN
+F 2 "" H 7400 4050 50  0001 C CNN
+F 3 "~" H 7400 4050 50  0001 C CNN
+	1    7200 4050
+	0    1    1    0
+$EndComp
+Wire Wire Line
+	6600 3950 7200 3950
+Wire Wire Line
+	6600 4050 7200 4050
 $EndSCHEMATC

Commit message: Updated footprints
Parts:
- C601: footprint (none) -> Capacitor_SMD:C_Elec_10x10.2
- C602: footprint C0603 -> Capacitor_SMD:C_0603_1608Metric
- J601: footprint (none) -> Connector_PinHeader_1.27mm:PinHeader_2x03_P1.27mm_Horizontal
- JP601: footprint (none) -> Jumper:SolderJumper-2_P1.3mm_Bridged_RoundedPad1.0x1.5mm
- R601, R602: footprint R0603 -> Resistor_SMD:R_0603_1608Metric
- TP601, TP602: footprint (none) -> TestPoint:TestPoint_Pad_1.5x1.5mm
Changed lines of the file:
@@
 F 0 "R601" H 5370 2796 50  0000 L CNN
 F 1 "10k" H 5370 2705 50  0000 L CNN
-F 2 "R0603" V 5230 2750 50  0001 C CNN
+F 2 "Resistor_SMD:R_0603_1608Metric" V 5230 2750 50  0001 C CNN
 F 3 "~" H 5300 2750 50  0001 C CNN
 F 4 "-SLAVE" H 5300 2750 50  0001 C CNN "Config"
@@
 F 0 "R602" H 6770 2796 50  0000 L CNN
 F 1 "10k" H 6770 2705 50  0000 L CNN
-F 2 "R0603" V 6630 2750 50  0001 C CNN
+F 2 "Resistor_SMD:R_0603_1608Metric" V 6630 2750 50  0001 C CNN
 F 3 "~" H 6700 2750 50  0001 C CNN
 F 4 "-SLAVE" H 6700 2750 50  0001 C CNN "Config"
@@
 F 0 "C602" H 5715 1946 50  0000 L CNN
 F 1 "100nF" H 5715 1855 50  0000 L CNN
-F 2 "C0603" H 5638 1750 50  0001 C CNN
+F 2 "Capacitor_SMD:C_0603_1608Metric" H 5638 1750 50  0001 C CNN
 F 3 "~" H 5600 1900 50  0001 C CNN
 F 4 "-SLAVE" H 5600 1900 50  0001 C CNN "Config"
@@
 F 0 "C601" H 5268 1946 50  0000 L CNN
 F 1 "22uF" H 5268 1855 50  0000 L CNN
-F 2 "" H 5188 1750 50  0001 C CNN
+F 2 "Capacitor_SMD:C_Elec_10x10.2" H 5188 1750 50  0001 C CNN
 F 3 "~" H 5150 1900 50  0001 C CNN
 F 4 "-SLAVE" H 5150 1900 50  0001 C CNN "Config"
@@
 F 0 "J601" H 9000 2975 50  0000 C CNN
 F 1 "Conn_02x03_Odd_Even" H 9000 2976 50  0001 C CNN
-F 2 "" H 8950 2750 50  0001 C CNN
+F 2 "Connector_PinHeader_1.27mm:PinHeader_2x03_P1.27mm_Horizontal" H 8950 2750 50  0001 C CNN
 F 3 "~" H 8950 2750 50  0001 C CNN
 F 4 "-SLAVE" H 8950 2750 50  0001 C CNN "Config"
@@
 F 0 "JP601" H 9500 2771 50  0000 C CNN
 F 1 "Jumper_NC_Small" H 9500 2771 50  0001 C CNN
-F 2 "" H 9500 2650 50  0001 C CNN
+F 2 "Jumper:SolderJumper-2_P1.3mm_Bridged_RoundedPad1.0x1.5mm" H 9500 2650 50  0001 C CNN
 F 3 "~" H 9500 2650 50  0001 C CNN
 	1    9500 2650
@@
 F 0 "TP601" V 7200 4138 50  0000 L CNN
 F 1 "uC-WiFi-Tx" V 7245 4138 50  0001 L CNN
-F 2 "" H 7400 3950 50  0001 C CNN
+F 2 "TestPoint:TestPoint_Pad_1.5x1.5mm" H 7400 3950 50  0001 C CNN
 F 3 "~" H 7400 3950 50  0001 C CNN
 	1    7200 3950
@@
 F 0 "TP602" V 7200 4238 50  0000 L CNN
 F 1 "uC-WiFi-Rx" V 7245 4238 50  0001 L CNN
-F 2 "" H 7400 4050 50  0001 C CNN
+F 2 "TestPoint:TestPoint_Pad_1.5x1.5mm" H 7400 4050 50  0001 C CNN
 F 3 "~" H 7400 4050 50  0001 C CNN
 	1    7200 4050

Commit message: Added motor footprint, made init pcb
Parts:
- J601: footprint Connector_PinHeader_1.27mm:PinHeader_2x03_P1.27mm_Horizontal -> Connector_PinHeader_1.27mm:PinHeader_2x03_P1.27mm_Vertical
- TP601, TP602: footprint TestPoint:TestPoint_Pad_1.5x1.5mm -> TestPoint:TestPoint_Pad_D2.0mm
- U601: symbol 24-clocks:ESP32-WROOM-32D -> 24-clocks-rescue:ESP32-WROOM-32D-24-clocks
Changed lines of the file:
@@
 $EndDescr
 $Comp
-L 24-clocks:ESP32-WROOM-32D U?
+L 24-clocks-rescue:ESP32-WROOM-32D-24-clocks U?
 U 1 1 5FDA8E5C
 P 6000 4150
@@
 F 0 "J601" H 9000 2975 50  0000 C CNN
 F 1 "Conn_02x03_Odd_Even" H 9000 2976 50  0001 C CNN
-F 2 "Connector_PinHeader_1.27mm:PinHeader_2x03_P1.27mm_Horizontal" H 8950 2750 50  0001 C CNN
+F 2 "Connector_PinHeader_1.27mm:PinHeader_2x03_P1.27mm_Vertical" H 8950 2750 50  0001 C CNN
 F 3 "~" H 8950 2750 50  0001 C CNN
 F 4 "-SLAVE" H 8950 2750 50  0001 C CNN "Config"
@@
 F 0 "TP601" V 7200 4138 50  0000 L CNN
 F 1 "uC-WiFi-Tx" V 7245 4138 50  0001 L CNN
-F 2 "TestPoint:TestPoint_Pad_1.5x1.5mm" H 7400 3950 50  0001 C CNN
+F 2 "TestPoint:TestPoint_Pad_D2.0mm" H 7400 3950 50  0001 C CNN
 F 3 "~" H 7400 3950 50  0001 C CNN
 	1    7200 3950
@@
 F 0 "TP602" V 7200 4238 50  0000 L CNN
 F 1 "uC-WiFi-Rx" V 7245 4238 50  0001 L CNN
-F 2 "TestPoint:TestPoint_Pad_1.5x1.5mm" H 7400 4050 50  0001 C CNN
+F 2 "TestPoint:TestPoint_Pad_D2.0mm" H 7400 4050 50  0001 C CNN
 F 3 "~" H 7400 4050 50  0001 C CNN
 	1    7200 4050
