File: hardware/pcb/24-c-com-bus.sch (KiCad schematic (older format))
At the start: 9 parts, among them J401 S4B_XH_SM4_TB, J402 S4B_XH_SM4_TB, U401 MAX3485

Commit message: Changed supply to 7V
Parts:
- D401: symbol SparkFun-DiscreteSemi:PESD1CAN -> 24-clocks-rescue:PESD1CAN-SparkFun-DiscreteSemi
Changed lines of the file:
@@
 EESchema Schematic File Version 4
-LIBS:24-clocks-cache
-EELAYER 29 0
+EELAYER 30 0
 EELAYER END
 $Descr A4 11693 8268
@@
 	4450 3150 5250 3150
 $Comp
-L SparkFun-DiscreteSemi:PESD1CAN D401
+L 24-clocks-rescue:PESD1CAN-SparkFun-DiscreteSemi D401
 U 1 1 5FEA3168
 P 6900 3550
+AR Path="/5FEA3168" Ref="D401"  Part="1"
+AR Path="/5FD135B5/5FEA3168" Ref="D401"  Part="1"
 F 0 "D401" V 6858 3778 45  0000 L CNN
 F 1 "PESD1CAN" V 6942 3778 45  0000 L CNN

Commit message: First placement
Connections:
- net +9V renamed +7.5V
Changed lines of the file:
@@
-	1    0    0    -1
-$EndComp
-$Comp
-L power:+9V #PWR?
-U 1 1 5FD2E217
-P 7450 1800
-AR Path="/5FD2E217" Ref="#PWR?"  Part="1"
-AR Path="/5FD135B5/5FD2E217" Ref="#PWR0402"  Part="1"
-F 0 "#PWR0402" H 7450 1650 50  0001 C CNN
-F 1 "+9V" H 7465 1973 50  0000 C CNN
-F 2 "" H 7450 1800 50  0001 C CNN
-F 3 "" H 7450 1800 50  0001 C CNN
-	1    7450 1800
 	1    0    0    -1
 $EndComp
@@
 	-1   0    0    -1
 $EndComp
-$Comp
-L power:+9V #PWR?
-U 1 1 5FD2E239
-P 6350 1800
-AR Path="/5FD2E239" Ref="#PWR?"  Part="1"
-AR Path="/5FD135B5/5FD2E239" Ref="#PWR0401"  Part="1"
-F 0 "#PWR0401" H 6350 1650 50  0001 C CNN
-F 1 "+9V" H 6365 1973 50  0000 C CNN
-F 2 "" H 6350 1800 50  0001 C CNN
-F 3 "" H 6350 1800 50  0001 C CNN
-	1    6350 1800
-	-1   0    0    -1
-$EndComp
 Wire Wire Line
 	6350 1800 6350 1850
@@
 Wire Wire Line
 	6900 3900 6900 3850
+$Comp
+L power:+7.5V #PWR0108
+U 1 1 6007755B
+P 6350 1800
+F 0 "#PWR0108" H 6350 1650 50  0001 C CNN
+F 1 "+7.5V" H 6365 1973 50  0000 C CNN
+F 2 "" H 6350 1800 50  0001 C CNN
+F 3 "" H 6350 1800 50  0001 C CNN
+	1    6350 1800
+	1    0    0    -1
+$EndComp
+$Comp
+L power:+7.5V #PWR0110
+U 1 1 60077F85
+P 7450 1800
+F 0 "#PWR0110" H 7450 1650 50  0001 C CNN
+F 1 "+7.5V" H 7465 1973 50  0000 C CNN
+F 2 "" H 7450 1800 50  0001 C CNN
+F 3 "" H 7450 1800 50  0001 C CNN
+	1    7450 1800
+	1    0    0    -1
+$EndComp
 $EndSCHEMATC

Commit message: Added caps to hall sensors
Parts:
- C401: Config -MASTER -> (none)
Changed lines of the file:
@@
 F 2 "Capacitor_SMD:C_0603_1608Metric" H 5088 3500 50  0001 C CNN
 F 3 "~" H 5050 3650 50  0001 C CNN
-F 4 "-MASTER" H 5050 3650 50  0001 C CNN "Config"
+F 4 "" H 5050 3650 50  0001 C CNN "Config"
 	1    5050 3650
 	1    0    0    -1
