File: hardware/pcb/24-clocks.sch (KiCad schematic (older format))
At the start: 37 parts

Commit message: Draft schematic (#1)
* Change schematic to hierarchical design

* Changed uC

* Created variants

* Added debug connector
Parts:
- removed BT?: BATTERY-20MM_SMD, BATTCON_20MM, symbol SparkFun-Batteries:BATTERY-20MM_SMD
- removed C? (x8): 100nF, C0603, symbol Device:C
- removed C? (x3): 22uF, symbol Device:CP
- removed J? (x2): Conn_01x04, symbol Connector_Generic:Conn_01x04
- removed J?: Conn_02x03_Odd_Even, symbol Connector_Generic:Conn_02x03_Odd_Even
- removed JP?: Jumper_NC_Small, symbol Device:Jumper_NC_Small
- removed R?: R, symbol Device:R
- removed R? (x5): 10k, R0603, symbol Device:R
- removed U?: MAX3485, symbol Interface_UART:MAX3485
- removed U?: VID66-08, TSOP-20, symbol 24-clocks:VID66-08
- removed U? (x2): VID28-05, symbol 24-clocks:VID28-05
- removed U?: AMS1117-5.0, Package_TO_SOT_SMD:SOT-223-3_TabPin2, symbol Regulator_Linear:AMS1117-5.0
- removed U?: AMS1117-3.3, Package_TO_SOT_SMD:SOT-223-3_TabPin2, symbol Regulator_Linear:AMS1117-3.3
- removed U? (x2): AH3572, Package_TO_SOT_SMD:SOT-23, symbol Sensor_Magnetic:SM351LT
- removed U?: DS1307+, Package_DIP:DIP-8_W7.62mm, symbol Timer_RTC:DS1307+
- removed U?: ESP32-WROOM-32D, RF_Module:ESP32-WROOM-32, symbol 24-clocks:ESP32-WROOM-32D
- removed U?: STM32L031K6Tx, Package_QFP:LQFP-32_7x7mm_P0.8mm, symbol MCU_ST_STM32L0:STM32L031K6Tx
- removed U?: 24LC512, symbol Memory_EEPROM:24LC512
- removed Y?: 32.768kHz, CRYSTAL-SMD-3.2X1.5MM, symbol SparkFun-Clocks:CRYSTAL-32.768KHZSMD-3.2X1.5
- gave numbers to parts that had none: 2
Connections:
- net labels removed: BOOT0, CWA, CWB, ESP-EN, ESP-IO0, ESP-RxD0, ESP-TxD0, GND, HAL-A, HAL-B, MA1, MA2, MA3, MA4, MB1, MB2, MB3, MB4, MRST, RCLK, RS485-A, RS485-B, RS485-DE, RS485-Rx, RS485-Tx, RST, STEPA, STEPB, SWDCLK, SWDIO, Serial-Rx, Serial-Tx, uC-Main-Rx, uC-Main-Tx
- wire segments 200 -> 26
- no-connect marks 1 -> 0
Other:
- moved on the sheet: R101, R102

Commit message: Updated footprints
Parts:
- R101, R102: footprint R0603 -> Resistor_SMD:R_0603_1608Metric
Changed lines of the file:
@@
 F 0 "R101" H 4420 5046 50  0000 L CNN
 F 1 "5k" H 4420 4955 50  0000 L CNN
-F 2 "R0603" V 4280 5000 50  0001 C CNN
+F 2 "Resistor_SMD:R_0603_1608Metric" V 4280 5000 50  0001 C CNN
 F 3 "~" H 4350 5000 50  0001 C CNN
 	1    4350 5000
@@
 F 0 "R102" H 4820 5046 50  0000 L CNN
 F 1 "5k" H 4820 4955 50  0000 L CNN
-F 2 "R0603" V 4680 5000 50  0001 C CNN
+F 2 "Resistor_SMD:R_0603_1608Metric" V 4680 5000 50  0001 C CNN
 F 3 "~" H 4750 5000 50  0001 C CNN
 	1    4750 5000

Commit message: Finished PCB (#3)
* Created PCB outline and first placement

* Changed connectors

* Minor

* Included all 3D files

* Mixed changes

* Changed supply to 7V

* Archived PCB project

* Update 24-clocks-rescue.lib

* First placement

* Routed supplies

* Update 24-clocks.kicad_pcb

* Added routing

* Routed more nets

* Finished routing

* Archived project

* Replace hash and date

* minor

* Update pcb.yml

* Update pcb.yml

* Update pcb.yml

* Update pcb.yml

* Auto update commit date and hash

* Update output

* changed outputs

* Added layer to output

* Update hash and date also in sch

* Added caps to hall sensors

* Cleanup files
Parts:
- added H101, H102, H103, H104: MountingHole, MountingHole:MountingHole_3.2mm_M3, symbol Mechanical:MountingHole
Changed lines of the file:
@@
 EESchema Schematic File Version 4
-LIBS:24-clocks-cache
-EELAYER 29 0
+EELAYER 30 0
 EELAYER END
 $Descr A4 11693 8268
@@
 Sheet 1 7
 Title "24 Clocks"
-Date "2020-12-06"
-Rev "V0.x"
+Date "GITDATE"
+Rev "GITHASH"
 Comp "Martin van Leussen"
 Comment1 ""
@@
 Comment4 ""
 $EndDescr
-$Comp
-L power:+9V #PWR0101
-U 1 1 5FC806BB
-P 1400 1850
-F 0 "#PWR0101" H 1400 1700 50  0001 C CNN
-F 1 "+9V" H 1415 2023 50  0000 C CNN
-F 2 "" H 1400 1850 50  0001 C CNN
-F 3 "" H 1400 1850 50  0001 C CNN
-	1    1400 1850
-	1    0    0    -1
-$EndComp
 $Comp
 L power:+5V #PWR0102
@@
 I2C-SDA
 $Sheet
-S 5400 1700 1750 3900
+S 5400 1700 1750 4000
 U 5FDEAABE
 F0 "uC" 50
@@
 F14 "I2C-SCL" O L 5400 5200 50
 F15 "I2C-SDA" B L 5400 5350 50
+F16 "RTC-CLK" I L 5400 5500 50
 $EndSheet
 $Sheet
@@
 F0 "Power Supply" 50
 F1 "24-c-supply.sch" 50
-F2 "+9V" I L 1750 1950 50
+F2 "+7V" I L 1750 1950 50
 F3 "+5V" O R 2900 1950 50
 F4 "+3V3" O R 2900 2300 50
@@
 $EndSheet
 $Sheet
-S 2600 4950 1100 650
+S 2600 4950 1100 750
 U 5FDBDABC
 F0 "RTC and Memory" 50
@@
 F2 "I2C-SDA" B R 3700 5350 50
 F3 "I2C-SCL" I R 3700 5200 50
+F4 "RTC-CLK" O R 3700 5500 50
 $EndSheet
 Wire Wire Line
@@
 Wire Wire Line
 	3700 5350 4750 5350
+$Comp
+L Mechanical:MountingHole H101
+U 1 1 5FEC3F65
+P 650 7000
+F 0 "H101" H 750 7046 50  0000 L CNN
+F 1 "MountingHole" H 750 6955 50  0000 L CNN
+F 2 "MountingHole:MountingHole_3.2mm_M3" H 650 7000 50  0001 C CNN
+F 3 "~" H 650 7000 50  0001 C CNN
+	1    650  7000
+	1    0    0    -1
+$EndComp
+$Comp
+L Mechanical:MountingHole H102
+U 1 1 5FEC5189
+P 650 7200
+F 0 "H102" H 750 7246 50  0000 L CNN
+F 1 "MountingHole" H 750 7155 50  0000 L CNN
+F 2 "MountingHole:MountingHole_3.2mm_M3" H 650 7200 50  0001 C CNN
+F 3 "~" H 650 7200 50  0001 C CNN
+	1    650  7200
+	1    0    0    -1
+$EndComp
+$Comp
+L Mechanical:MountingHole H103
+U 1 1 5FEC5459
+P 650 7400
+F 0 "H103" H 750 7446 50  0000 L CNN
+F 1 "MountingHole" H 750 7355 50  0000 L CNN
+F 2 "MountingHole:MountingHole_3.2mm_M3" H 650 7400 50  0001 C CNN
+F 3 "~" H 650 7400 50  0001 C CNN
+	1    650  7400
+	1    0    0    -1
+$EndComp
+$Comp
+L Mechanical:MountingHole H104
+U 1 1 5FEC567F
+P 650 7600
+F 0 "H104" H 750 7646 50  0000 L CNN
+F 1 "MountingHole" H 750 7555 50  0000 L CNN
+F 2 "MountingHole:MountingHole_3.2mm_M3" H 650 7600 50  0001 C CNN
+F 3 "~" H 650 7600 50  0001 C CNN
+	1    650  7600
+	1    0    0    -1
+$EndComp
+$Comp
+L power:+7.5V #PWR0101
+U 1 1 60073D60
+P 1400 1850
+F 0 "#PWR0101" H 1400 1700 50  0001 C CNN
+F 1 "+7.5V" H 1415 2023 50  0000 C CNN
+F 2 "" H 1400 1850 50  0001 C CNN
+F 3 "" H 1400 1850 50  0001 C CNN
+	1    1400 1850
+	1    0    0    -1
+$EndComp
+Wire Wire Line
+	3700 5500 5400 5500
 $EndSCHEMATC
